File: MainBoard.kicad_pcb (KiCad board)
At the start: 4 copper layers, 150 x 100 mm, 89 parts, among them J4 Conn_01x06_Pin, J7 IEC61076-2_M8_B-coding_01x03_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, SW2 PBH2UEESNPNAGX, U1 STM32H723ZGT6, U4 CA-IS2062W, U51 24AA02-OT, Y5 12M, Y6 32,768kHz

Commit message: DC_DC_blocks + layout
Parts:
- removed C14: 10n, Capacitor_SMD:C_0603_1608Metric
- removed R4, R5: 62R, Resistor_SMD:R_0603_1608Metric
- removed SW2: PBH2UEESNPNAGX, E-M-Electromechanics:PBH2UEESNPNAGX
- removed TP10: FAN2_DRV, TestPoint:TestPoint_Pad_D1.5mm
- removed TP22: I2C2.SCK, TestPoint:TestPoint_Pad_D1.5mm
- removed TP23: I2C2.DATA, TestPoint:TestPoint_Pad_D1.5mm
- added C133: 10u/25V/X5R, Capacitor_SMD:C_0805_2012Metric, F.Cu at (88.8, 84.0)
- added C134: 10u/25V/X5R, Capacitor_SMD:C_0805_2012Metric, F.Cu at (78.0, 107.8)
- added C135: 22n/X7R, Capacitor_SMD:C_0603_1608Metric, F.Cu at (93.3, 85.8)
- added C136: 22n/X7R, Capacitor_SMD:C_0603_1608Metric, F.Cu at (75.9, 106.2)
- added C137: 100p, Capacitor_SMD:C_0603_1608Metric, F.Cu at (76.9, 92.8)
- added C138: 100p, Capacitor_SMD:C_0603_1608Metric, F.Cu at (93.0, 103.6)
- added C139: 22u/16V/X7R, Capacitor_SMD:C_0805_2012Metric, F.Cu at (68.6, 90.8)
- added C140: 22u/16V/X7R, Capacitor_SMD:C_0805_2012Metric, F.Cu at (99.5, 102.1)
- added C141: 22u/16V/X7R, Capacitor_SMD:C_0805_2012Metric, F.Cu at (70.8, 90.8)
- added C142: 22u/16V/X7R, Capacitor_SMD:C_0805_2012Metric, F.Cu at (97.3, 102.1)
- added C143: 22u/16V/X7R, Capacitor_SMD:C_0805_2012Metric, F.Cu at (73.1, 90.8)
- added C144: 22u/16V/X7R, Capacitor_SMD:C_0805_2012Metric, F.Cu at (95.1, 102.1)
- added C149: 100p, Capacitor_SMD:C_0603_1608Metric, F.Cu at (82.2, 91.1)
- added C150: 2n2, Capacitor_SMD:C_0603_1608Metric, F.Cu at (80.4, 92.7)
- added C151: 10u/25V/X5R, Capacitor_SMD:C_0805_2012Metric, F.Cu at (88.8, 81.7)
- added C152: 2n2, Capacitor_SMD:C_0603_1608Metric, F.Cu at (87.7, 100.2)
- added C153: 100p, Capacitor_SMD:C_0603_1608Metric, F.Cu at (87.8, 103.6)
- added C154: 0u22, Capacitor_SMD:C_0603_1608Metric, F.Cu at (91.4, 99.1)
- added C155: 0u1, Capacitor_SMD:C_0603_1608Metric, F.Cu at (75.1, 89.5)
- added IC3: RT8293BHZSP, E-M-IntegratedCircuits:SOIC127P600X175-9N, F.Cu at (78.6, 99.9)
- added IC4: RT8293BHZSP, E-M-IntegratedCircuits:SOIC127P600X175-9N, F.Cu at (88.6, 93.2)
- added L12: 6u8/5A, Inductor_SMD:L_APV_APH0850, F.Cu at (70.4, 100.6)
- added L13: 4u7/5A, Inductor_SMD:L_APV_APH0850, F.Cu at (96.1, 92.4)
- added L15: 1u/5A, Inductor_SMD:L_APV_APH0650, F.Cu at (89.2, 76.4)
- added R144: 62k, Resistor_SMD:R_0603_1608Metric, F.Cu at (78.7, 92.8)
- added R145: 11k8, Resistor_SMD:R_0603_1608Metric, F.Cu at (76.9, 88.5)
- added R146: 75k, Resistor_SMD:R_0603_1608Metric, F.Cu at (91.2, 103.6)
- added R147: 24k, Resistor_SMD:R_0603_1608Metric, F.Cu at (85.7, 98.9)
- added R148: 100k, Resistor_SMD:R_0603_1608Metric, F.Cu at (83.4, 104.7)
- added R149: 100k, Resistor_SMD:R_0603_1608Metric, F.Cu at (89.6, 99.1)
- added R150: 33k, Resistor_SMD:R_0603_1608Metric, F.Cu at (80.4, 89.4)
- added R151: 22k, Resistor_SMD:R_0603_1608Metric, F.Cu at (89.4, 103.6)
Connections:
- net /CANinterface/CAN_SH renamed /PowertrainInterface/CAN_SH
- C269 pad 1: Net-(U1PortG_PORTH-PC15) -> unconnected-(C269-Pad1)
- C270 pad 1: Net-(U1PortG_PORTH-PC14) -> unconnected-(C270-Pad1)
- U1 pad 1: /DiffGPS+IMU_modul/SPI.SCK -> unconnected-(U1PortE_PortF-PE2-Pad1)
- U1 pad 10: /MCU/I2C2.DATA -> unconnected-(U1PortE_PortF-PF0-Pad10)
- U1 pad 101: /MCU/USB_PD_ALERT -> unconnected-(U1PortA_PortB-PA9-Pad101)
- U1 pad 102: /MCU/USB_PD_RST -> unconnected-(U1PortA_PortB-PA10-Pad102)
- U1 pad 103: /MCU/USB_N -> unconnected-(U1PortA_PortB-PA11-Pad103)
- U1 pad 104: /MCU/USB_P -> unconnected-(U1PortA_PortB-PA12-Pad104)
- U1 pad 11: /MCU/I2C2.SCK -> unconnected-(U1PortE_PortF-PF1-Pad11)
- U1 pad 110: /SerialInterfaces/RS485-1.DTS -> unconnected-(U1PortA_PortB-PA15(JTDI)-Pad110)
- U1 pad 111: /SerialInterfaces/RS485-1.ucRX -> unconnected-(U1PortC_PortD-PC10-Pad111)
- U1 pad 112: /SerialInterfaces/RS485-1.ucTX -> unconnected-(U1PortC_PortD-PC11-Pad112)
- U1 pad 113: /SerialInterfaces/RS485-2.ucTX -> unconnected-(U1PortC_PortD-PC12-Pad113)
- U1 pad 114: /CANinterface/CAN1.RX -> unconnected-(U1PortC_PortD-PD0-Pad114)
- U1 pad 115: /CANinterface/CAN1.TX -> unconnected-(U1PortC_PortD-PD1-Pad115)
- U1 pad 116: /SerialInterfaces/RS485-2.ucRX -> unconnected-(U1PortC_PortD-PD2-Pad116)
- U1 pad 117: /MCU/HS-UART.CTS -> unconnected-(U1PortC_PortD-PD3-Pad117)
- U1 pad 118: /MCU/HS-UART.RTS -> unconnected-(U1PortC_PortD-PD4-Pad118)
- U1 pad 119: /MCU/HS-UART.TX -> unconnected-(U1PortC_PortD-PD5-Pad119)
- U1 pad 122: /MCU/HS-UART.RX -> unconnected-(U1PortC_PortD-PD6-Pad122)
- U1 pad 123: /MCU/X-SPI.RX-DATA -> unconnected-(U1PortC_PortD-PD7-Pad123)
- U1 pad 125: /MCU/X-SPI.RX-~{SS} -> unconnected-(U1PortG_PORTH-PG10-Pad125)
- U1 pad 126: Net-(RN3-R4.1) -> unconnected-(U1PortG_PORTH-PG11-Pad126)
- U1 pad 128: Net-(RN3-R3.1) -> unconnected-(U1PortG_PORTH-PG13-Pad128)
- U1 pad 129: Net-(RN3-R2.1) -> unconnected-(U1PortG_PORTH-PG14-Pad129)
- U1 pad 133: /MCU/X-SPI.RX-CLK -> unconnected-(U1PortA_PortB-PB3(JTDO-Pad133)
- U1 pad 135: /CANinterface/CAN2.RX -> unconnected-(U1PortA_PortB-PB5-Pad135)
- U1 pad 136: /CANinterface/CAN2.TX -> unconnected-(U1PortA_PortB-PB6-Pad136)
- U1 pad 137: /MCU/I2C1.DATA -> unconnected-(U1PortA_PortB-PB7-Pad137)
- U1 pad 139: /MCU/I2C1.CLK -> unconnected-(U1PortA_PortB-PB8-Pad139)
- U1 pad 141: /DiffGPS+IMU_modul/SPI.~{CS1} -> unconnected-(U1PortE_PortF-PE0-Pad141)
- U1 pad 142: /DiffGPS+IMU_modul/SPI.~{CS2} -> unconnected-(U1PortE_PortF-PE1-Pad142)
- U1 pad 18: /CANinterface/CAN3.RX -> unconnected-(U1PortE_PortF-PF6-Pad18)
- U1 pad 19: /CANinterface/CAN3.TX -> unconnected-(U1PortE_PortF-PF7-Pad19)
- U1 pad 2: /DiffGPS+IMU_modul/SPI.~{CS3} -> unconnected-(U1PortE_PortF-PE3-Pad2)
- U1 pad 26: /MCU/BATT_RST -> unconnected-(U1PortC_PortD-PC0-Pad26)
- U1 pad 27: /EtherNET_interface/RMII.MDC -> unconnected-(U1PortC_PortD-PC1-Pad27)
- U1 pad 3: /DiffGPS+IMU_modul/SPI.~{CS4} -> unconnected-(U1PortE_PortF-PE4-Pad3)
- U1 pad 35: /EtherNET_interface/RMII.~{INT}/REF_CLKO -> unconnected-(U1PortA_PortB-PA1-Pad35)
- U1 pad 36: /EtherNET_interface/RMII.MDIO -> unconnected-(U1PortA_PortB-PA2-Pad36)
- U1 pad 37: /AnalogIO/AnIN4 -> unconnected-(U1PortA_PortB-PA3-Pad37)
- U1 pad 4: /DiffGPS+IMU_modul/SPI.MISO -> unconnected-(U1PortE_PortF-PE5-Pad4)
- U1 pad 40: /AnalogIO/AnOUT1 -> unconnected-(U1PortA_PortB-PA4-Pad40)
- U1 pad 41: /AnalogIO/AnOUT2 -> unconnected-(U1PortA_PortB-PA5-Pad41)
- U1 pad 42: /AnalogIO/AnIN2 -> unconnected-(U1PortA_PortB-PA6-Pad42)
- U1 pad 43: /EtherNET_interface/RMII.CRS_DV -> unconnected-(U1PortA_PortB-PA7-Pad43)
- U1 pad 44: /EtherNET_interface/RMII.RXD0 -> unconnected-(U1PortC_PortD-PC4-Pad44)
- U1 pad 45: /EtherNET_interface/RMII.RXD1 -> unconnected-(U1PortC_PortD-PC5-Pad45)
- U1 pad 46: /EtherNET_interface/RMII.~{RST} -> unconnected-(U1PortA_PortB-PB0-Pad46)
- U1 pad 47: /AnalogIO/AnIN3 -> unconnected-(U1PortA_PortB-PB1-Pad47)
- U1 pad 49: /AnalogIO/AnIN1 -> unconnected-(U1PortE_PortF-PF11-Pad49)
- U1 pad 5: /DiffGPS+IMU_modul/SPI.MOSI -> unconnected-(U1PortE_PortF-PE6-Pad5)
- U1 pad 50: /MCU/I2C4.INT1 -> unconnected-(U1PortE_PortF-PF12-Pad50)
- U1 pad 53: /MCU/I2C4.INT2 -> unconnected-(U1PortE_PortF-PF13-Pad53)
- U1 pad 54: /MCU/I2C4.SCK -> unconnected-(U1PortE_PortF-PF14-Pad54)
- U1 pad 55: /MCU/I2C4.DATA -> unconnected-(U1PortE_PortF-PF15-Pad55)
- U1 pad 56: /SerialInterfaces/RS422.ucRX -> unconnected-(U1PortG_PORTH-PG0-Pad56)
- U1 pad 57: /SerialInterfaces/RS422.ucTX -> unconnected-(U1PortG_PORTH-PG1-Pad57)
- U1 pad 58: /SerialInterfaces/RS485-3.ucRX -> unconnected-(U1PortE_PortF-PE7-Pad58)
- U1 pad 59: /SerialInterfaces/RS485-3.ucTX -> unconnected-(U1PortE_PortF-PE8-Pad59)
- U1 pad 60: /SerialInterfaces/RS485-3.DTS -> unconnected-(U1PortE_PortF-PE9-Pad60)
- U1 pad 63: /MCU/LDO_Diasable -> unconnected-(U1PortE_PortF-PE10-Pad63)
- U1 pad 64: /MCU/CHARGE_Disable -> unconnected-(U1PortE_PortF-PE11-Pad64)
- U1 pad 65: /MCU/~{LED_SW_ON} -> unconnected-(U1PortE_PortF-PE12-Pad65)
- U1 pad 66: /DigitalIO/CSTOP1 -> unconnected-(U1PortE_PortF-PE13-Pad66)
- U1 pad 67: /DigitalIO/CSTOP2 -> unconnected-(U1PortE_PortF-PE14-Pad67)
- U1 pad 68: /EtherNET_interface/PoE_PSE/~{PoE_EN} -> unconnected-(U1PortE_PortF-PE15-Pad68)
- U1 pad 69: /Dual_FAN_ctrl/FAN1_feedback -> unconnected-(U1PortA_PortB-PB10-Pad69)
- U1 pad 70: /Dual_FAN_ctrl/FAN2_feedback -> unconnected-(U1PortA_PortB-PB11-Pad70)
- U1 pad 73: /MCU/X-SPI.TX-~{SS} -> unconnected-(U1PortA_PortB-PB12-Pad73)
- U1 pad 74: /MCU/X-SPI.TX-CLK -> unconnected-(U1PortA_PortB-PB13-Pad74)
- U1 pad 76: /MCU/X-SPI.TX-DATA -> unconnected-(U1PortA_PortB-PB15-Pad76)
- U1 pad 77: /SerialInterfaces/RS232.ucTX -> unconnected-(U1PortC_PortD-PD8-Pad77)
- U1 pad 78: /SerialInterfaces/RS232.ucRX -> unconnected-(U1PortC_PortD-PD9-Pad78)
- U1 pad 8: Net-(U1PortG_PORTH-PC14) -> unconnected-(U1PortG_PORTH-PC14-Pad8)
- U1 pad 81: /DigitalIO/OUT1 -> unconnected-(U1PortC_PortD-PD12-Pad81)
- U1 pad 82: /DigitalIO/OUT2 -> unconnected-(U1PortC_PortD-PD13-Pad82)
- U1 pad 85: /DigitalIO/OUT3 -> unconnected-(U1PortC_PortD-PD14-Pad85)
- U1 pad 86: /DigitalIO/OUT4 -> unconnected-(U1PortC_PortD-PD15-Pad86)
- U1 pad 9: Net-(U1PortG_PORTH-PC15) -> unconnected-(U1PortG_PORTH-PC15-Pad9)
- U1 pad 90: /DigitalIO/IN1 -> unconnected-(U1PortG_PORTH-PG5-Pad90)
- U1 pad 91: /DigitalIO/IN2 -> unconnected-(U1PortG_PORTH-PG6-Pad91)
- U1 pad 92: /DigitalIO/IN3 -> unconnected-(U1PortG_PORTH-PG7-Pad92)
- U1 pad 93: /DigitalIO/IN4 -> unconnected-(U1PortG_PORTH-PG8-Pad93)
- U1 pad 96: /Dual_FAN_ctrl/FAN1_drive -> unconnected-(U1PortC_PortD-PC6-Pad96)
- U1 pad 97: /Dual_FAN_ctrl/FAN2_drive -> unconnected-(U1PortC_PortD-PC7-Pad97)
- U1 pad 98: /SerialInterfaces/RS485-2.DTS -> unconnected-(U1PortC_PortD-PC8-Pad98)
- Y6 pad 1: Net-(U1PortG_PORTH-PC15) -> unconnected-(Y6-Pad1)
- Y6 pad 2: Net-(U1PortG_PORTH-PC14) -> unconnected-(Y6-Pad2)
Routing:
- net (no net): track 0.00 -> 71.2 mm, vias 0 -> 2
- net Net-(IC4-VIN): track 0.00 -> 27.5 mm, vias 0 -> 2
- net Net-(IC4-SW): track 0.00 -> 23.6 mm, vias 0 -> 4
- net unconnected-(U1PortA_PortB-PA9-Pad101): track 0.00 -> 20.9 mm, vias 0 -> 2
- net /MCU/USB_PD_ALERT: track 20.9 -> 0.00 mm, vias 2 -> 0
- net unconnected-(U1PortA_PortB-PA10-Pad102): track 0.00 -> 18.9 mm, vias 0 -> 2
- net /MCU/USB_PD_RST: track 18.9 -> 0.00 mm, vias 2 -> 0
- net Net-(R4-Pad2): track 18.7 -> 0.00 mm, vias 1 -> 0
- net Net-(IC4-FB): track 0.00 -> 17.0 mm
- net Net-(R5-Pad2): track 15.7 -> 0.00 mm, vias 1 -> 0
- net +5V: track 0.00 -> 15.6 mm, vias 0 -> 9
- net Net-(IC3-SW): track 0.00 -> 10.8 mm, vias 0 -> 5
- net GND: track 22.9 -> 32.1 mm, vias 71 -> 114
- net unconnected-(U1PortC_PortD-PC7-Pad97): track 0.00 -> 8.87 mm, vias 0 -> 1
- net /Dual_FAN_ctrl/FAN2_drive: track 8.87 -> 0.00 mm, vias 1 -> 0
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- added copper zone on F.Cu, net +3.3V
- added copper zone on F.Cu, net +5V
- added copper zone on In1.Cu, net +5V

Commit message: UPB_PD block + Layout
Parts:
- added C108: 1u/16V/X7R, Capacitor_SMD:C_0805_2012Metric, F.Cu at (191.1, 100.7)
- added C109: 1u/16V/X7R, Capacitor_SMD:C_0805_2012Metric, F.Cu at (186.8, 100.7)
- added C110: 1u/16V/X7R, Capacitor_SMD:C_0805_2012Metric, F.Cu at (180.4, 101.7)
- added C111: C, Capacitor_SMD:C_0805_2012Metric, F.Cu at (195.1, 100.7)
- added C112: 4u7/X7R/50V, Capacitor_SMD:C_1210_3225Metric, F.Cu at (171.3, 116.3)
- added C113: 0u1, Capacitor_SMD:C_0603_1608Metric, F.Cu at (177.8, 112.9)
- added D27: ??V/0.5W, Diode_SMD:D_SOD-123F, F.Cu at (184.5, 101.2)
- added D28: ESDA25W, Package_TO_SOT_SMD:SOT-323_SC-70, F.Cu at (184.3, 116.8)
- added D29: P4SMAJ28A, Diode_SMD:D_SMA, F.Cu at (170.2, 120.2)
- added D30: P4SMAJ28A, Diode_SMD:D_SMA, F.Cu at (166.1, 110.1)
- added IC2: STUSB4500LQTR, Package_DFN_QFN:QFN-24-1EP_4x4mm_P0.5mm_EP2.7x2.7mm, F.Cu at (187.8, 108.3)
- added J15: USB_C_2.0, Connector_USB:USB_C_Receptacle_GCT_USB4110-GF-A, F.Cu at (181.3, 127.3)
- added Q6: STL9P3LLH6, Package_SON:Diodes_PowerDI3333-8, F.Cu at (173.9, 111.6)
- added Q7: STL9P3LLH6, Package_SON:Diodes_PowerDI3333-8, F.Cu at (173.3, 104.9)
- added R111: 1M, Resistor_SMD:R_0805_2012Metric, F.Cu at (188.3, 119.4)
- added R116: 100k, Resistor_SMD:R_0603_1608Metric, F.Cu at (190.1, 114.4)
- added R117: 100k, Resistor_SMD:R_0603_1608Metric, F.Cu at (188.9, 100.5)
- added R118: 10k, Resistor_SMD:R_0603_1608Metric, F.Cu at (186.4, 114.4)
- added R119: 470R, Resistor_SMD:R_0603_1608Metric, F.Cu at (182.3, 101.9)
- added R120: 1k, Resistor_SMD:R_0603_1608Metric, F.Cu at (194.4, 106.4)
- added R121: 100k, Resistor_SMD:R_0603_1608Metric, F.Cu at (192.8, 114.4)
- added R122: 22k, Resistor_SMD:R_0603_1608Metric, F.Cu at (192.8, 110.1)
- added R123: 100, Resistor_SMD:R_0603_1608Metric, F.Cu at (177.8, 114.7)
- added R124: 4k7, Resistor_SMD:R_0603_1608Metric, F.Cu at (193.1, 100.5)
- added R125: 1k, Resistor_SMD:R_0603_1608Metric, F.Cu at (188.2, 114.4)
- added TP11: VBUS_USB, TestPoint:TestPoint_THTPad_D1.5mm_Drill0.7mm, F.Cu at (196.7, 109.6)
- added TP22: I2C2.SCK, TestPoint:TestPoint_Pad_D1.5mm, F.Cu at (184.2, 95.6)
- added TP23: I2C2.DATA, TestPoint:TestPoint_Pad_D1.5mm, F.Cu at (184.2, 92.6)
- added U27: USBLC6-2P6, Package_TO_SOT_SMD:SOT-666, F.Cu at (181.3, 119.6)
Routing:
- net /USB_PD/VBUS_USB: track 0.00 -> 41.5 mm, vias 0 -> 10
- net (no net): track 71.2 -> 33.4 mm, vias 2 -> 4
- net Net-(D27-K): track 0.00 -> 24.9 mm, vias 0 -> 2
- net /USB_PD/USB_N: track 0.00 -> 24.1 mm
- net /USB_PD/USB_P: track 0.00 -> 23.5 mm
- net /USB_PD/CC1_USB: track 0.00 -> 22.7 mm, vias 0 -> 2
- net /USB_PD/USB_PD_ALERT: track 0.00 -> 21.4 mm, vias 0 -> 1
- net GND: track 32.1 -> 52.4 mm, vias 114 -> 158
- net /USB_PD/CC2_USB: track 0.00 -> 19.7 mm
- net /USB_PD/USB_PD_RST: track 0.00 -> 18.9 mm, vias 0 -> 1
- net /USB_PD/I2C2.DATA: track 0.00 -> 18.6 mm, vias 0 -> 1
- net Net-(R121-Pad2): track 0.00 -> 17.9 mm, vias 0 -> 2
- net /USB_PD/I2C2.SCK: track 0.00 -> 16.2 mm, vias 0 -> 1
- net Net-(IC2-ADDR0): track 0.00 -> 11.9 mm, vias 0 -> 2
- net +5V: track 15.6 -> 26.3 mm, vias 9 -> 24
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- added copper zone on B.Cu, net /USB_PD/VBUS_USB
- added copper zone on F.Cu, net /USB_PD/VBUS_USB
