File: HumanInterfaceCircuits.kicad_sch (KiCad schematic)
At the start: 0 parts

Commit message: added schematic for input (switch, PAS, analog) + output
Parts:
- added C1: 470nF, symbol Device:C
- added D1: 1N4148W, PCM_JLCPCB:D_SOD-123, symbol PCM_JLCPCB-Diodes:Switching,1N4148W
- added R1: 1K2, symbol Device:R
- added R2: 33k, symbol Device:R
- added R3: 10k, symbol Device:R
Connections:
- new net +12V: R1.1
- new net +3.3V: D1.1
- new net GND: C1.2, R3.2
- new net MCU_SW: C1.1, D1.2, R2.2, R3.1
- new net SW: R1.2, R2.1
Other:
- note added: "Rth = R3//(R2+R1) = 7.7 k C = 1 / (2*pi × 50Hz × Rth) = 470nF"
- note added: "V_MCUmax = Vccmax * R3/(R1+R2+R2)=3V2 @ 14V for Vccmax V_MCUmin = Vccmin * R3/(R1+R2+R2)=2.3V @ 10V for Vccmin"
- note added: "also do debouce in software (20ms steady state)"
- note added: "wetting current of 10mA 12V/0.01A=1k2"

Commit message: wiring MCU to input and ouput
Changed lines of the file:
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@@
 	)
 	(hierarchical_label "MCU_SW"
-		(shape input)
+		(shape output)
 		(at 95.25 72.39 0)
 		(effects
