File: HumanInterfaceCircuits.kicad_sch (KiCad schematic)
At the start: 0 parts

Commit message: I/O Schematic rebuild from DRAFT by Nathann
Parts:
- added C87, C88, C89, C90, C91, C92, C93, C96, C97, C98, C99: 470nF, symbol Device:C
- added D23, D24, D25, D26, D33, D34, D35, D36, D37, D38, D39: 1N4148W, PCM_JLCPCB:D_SOD-123, symbol PCM_JLCPCB-Diodes:Switching,1N4148W
- added J18: (no value), symbol higo:Z509BM_C_04_00_0000
- added J21: (no value), symbol higo:Z809FM_C_04_00_0000
- added R100, R103, R106, R109, R127, R130, R133, R136, R139, R92, R97: 1.2kΩ, PCM_JLCPCB:R_0805, symbol PCM_JLCPCB-Resistors:0805,1.2kΩ
- added R101, R104, R107, R110, R128, R131, R134, R137, R94, R95, R98: 10kΩ, PCM_JLCPCB:R_0805, symbol PCM_JLCPCB-Resistors:0805,10kΩ
- added R102, R105, R108, R112, R129, R132, R135, R138, R93, R96, R99: 33kΩ, PCM_JLCPCB:R_0805, symbol PCM_JLCPCB-Resistors:0805,33kΩ
Connections:
- new net: J21.3, R108.1, R109.2
- new net: J18.2, R92.2, R93.1
- new net: J18.3, R96.1, R97.2
- new net: J18.4, R100.2, R99.1
- new net: J18.5, R102.1, R103.2
- new net: J21.5, R129.1, R130.2
- new net: J21.7, R135.1, R136.2
- new net: J21.2, R105.1, R106.2
- new net: J21.4, R112.1, R127.2
- new net: J21.6, R132.1, R133.2
- new net: J21.8, R138.1, R139.2
- new net +12V: R100.1, R103.1, R106.1, R109.1, R127.1, R130.1, R133.1, R136.1, R139.1, R92.1, R97.1
- new net +3.3V: D23.1, D24.1, D25.1, D26.1, D33.1, D34.1, D35.1, D36.1, D37.1, D38.1, D39.1
- new net GND: C87.2, C88.2, C89.2, C90.2, C91.2, C92.2, C93.2, C96.2, C97.2, C98.2, C99.2, J18.1, J21.1, R101.2, R104.2, R107.2, R110.2, R128.2, R131.2, R134.2, R137.2, R94.2, R95.2, R98.2
- new net MCU_SW: C87.1, C88.1, C89.1, C90.1, C91.1, C92.1, C93.1, C96.1, C97.1, C98.1, C99.1, D23.2, D24.2, D25.2, D26.2, D33.2, D34.2, D35.2, D36.2, D37.2, D38.2, D39.2, R101.1, R102.2, R104.1, R105.2, R107.1, R108.2, R110.1, R112.2, R128.1, R129.2, R131.1, R132.2, R134.1, R135.2, R137.1, R138.2, R93.2, R94.1, R95.1, R96.2, R98.1, R99.2
Other:
- note added: "Rth = R3//(R2+R1) = 7.7 k C = 1 / (2*pi × 50Hz × Rth) = 470nF"
- note added: "V_MCUmax = Vccmax * R3/(R1+R2+R2)=3V2 @ 14V for Vccmax V_MCUmin = Vccmin * R3/(R1+R2+R2)=2.3V @ 10V for Vccmin"
- note added: "also do debouce in software (20ms steady state)"
- note added: "drive commodo"
- note added: "lightning commodo"
- note added: "wetting current of 10mA 12V/0.01A=1k2"

Commit message: integration of commodo signals to design
Connections:
- net SpeedLimSW_IN: now reaches J21.3, R108.1, R109.2
- net DirIndSW_L_IN: now reaches J18.2, R92.2, R93.1
- net DirIndSW_R_IN: now reaches J18.3, R96.1, R97.2
- net AcousticWarnSW_IN: now reaches J18.4, R100.2, R99.1
- net LightChangeSW_IN: now reaches J18.5, R102.1, R103.2
- net ForwardSW_IN: now reaches J21.5, R129.1, R130.2
- net Assist-SW_IN: now reaches J21.7, R135.1, R136.2
- net MappingSW_IN: now reaches J21.2, R105.1, R106.2
- net ReverseSW_IN: now reaches J21.4, R112.1, R127.2
- net Assist+SW_IN: now reaches J21.6, R132.1, R133.2
- net VehicleStartSW_IN: now reaches J21.8, R138.1, R139.2
- removed net MCU_SW: C87.1, C88.1, C89.1, C90.1, C91.1, C92.1, C93.1, C96.1, C97.1, C98.1, C99.1, D23.2, D24.2, D25.2, D26.2, D33.2, D34.2, D35.2, D36.2, D37.2, D38.2, D39.2, R101.1, R102.2, R104.1, R105.2, R107.1, R108.2, R110.1, R112.2, R128.1, R129.2, R131.1, R132.2, R134.1, R135.2, R137.1, R138.2, R93.2, R94.1, R95.1, R96.2, R98.1, R99.2
- new net AcousticWarnSW: C89.1, D25.2, R98.1, R99.2
- new net Assist+SW: C97.1, D37.2, R131.1, R132.2
- new net Assist-SW: C98.1, D38.2, R134.1, R135.2
- new net DirIndSW_L: C87.1, D23.2, R93.2, R94.1
- new net DirIndSW_R: C88.1, D24.2, R95.1, R96.2
- new net ForwardSW: C96.1, D36.2, R128.1, R129.2
- new net LightChangeSW: C90.1, D26.2, R101.1, R102.2
- new net MappingSW: C91.1, D33.2, R104.1, R105.2
- new net ReverseSW: C93.1, D35.2, R110.1, R112.2
- new net SpeedLimSW: C92.1, D34.2, R107.1, R108.2
- new net VehicleStartSW: C99.1, D39.2, R137.1, R138.2
Other:
- note added: "Left direction indicator Right direction indicator Acoustic warning (if I recall) Light change (toggle between driving and passing lights)"
- note added: "Mapping button Speed limiter start/stop Reverse Foward (the two arrow) Assist + Assist - Vehicule start"
Changed lines of the file:
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@@
+		)
+	)
+	(text "Mapping button\nSpeed limiter start/stop\nReverse\nFoward (the two arrow)\nAssist +\nAssist -\nVehicule start"
+		(exclude_from_sim no)
+		(at 253.492 147.828 0)
+		(effects
+			(font
+				(size 1.27 1.27)
+			)
+			(justify left)
 		)
 	)
@@
 		)
 	)
+	(text "Left direction indicator\nRight direction indicator\nAcoustic warning (if I recall)\nLight change (toggle between driving and passing lights)"
+		(exclude_from_sim no)
+		(at 288.29 58.928 0)
+		(effects
+			(font
+				(size 1.27 1.27)
+			)
+			(justify left)
+		)
+	)
 	(junction
 		(at 214.63 64.77)
@@
 		)
 	)
-	(hierarchical_label "MCU_SW"
+	(label "SpeedLimSW_IN"
+		(at 218.44 86.36 0)
+		(effects
+			(font
+				(size 1.27 1.27)
+			)
+			(justify left bottom)
+		)
+	)
+	(label "LightChangeSW_IN"
+		(at 229.87 64.77 0)
+		(effects
+			(font
+				(size 1.27 1.27)
+			)
+			(justify left bottom)
+		)
+	)
+	(label "MappingSW_IN"
+		(at 218.44 83.82 0)
+		(effects
+			(font
+				(size 1.27 1.27)
+			)
+			(justify left bottom)
+		)
+	)
+	(label "VehicleStartSW_IN"
+		(at 214.63 162.56 0)
+		(effects
+			(font
+				(size 1.27 1.27)
+			)
+			(justify left bottom)
+		)
+	)
+	(label "ForwardSW_IN"
+		(at 214.63 156.21 0)
+		(effects
+			(font
+				(size 1.27 1.27)
+			)
+			(justify left bottom)
+		)
+	)
+	(label "DirIndSW_R_IN"
+		(at 229.87 59.69 0)
+		(effects
+			(font
+				(size 1.27 1.27)
+			)
+			(justify left bottom)
+		)
+	)
+	(label "Assist+SW_IN"
+		(at 214.63 160.02 0)
+		(effects
+			(font
+				(size 1.27 1.27)
+			)
+			(justify left bottom)
+		)
+	)
+	(label "Assist-SW_IN"
+		(at 214.63 137.16 0)
+		(effects
+			(font
+				(size 1.27 1.27)
+			)
+			(justify left bottom)
+		)
+	)
+	(label "DirIndSW_L_IN"
+		(at 233.68 57.15 0)
+		(effects
+			(font
+				(size 1.27 1.27)
+			)
+			(justify left bottom)
+		)
+	)
+	(label "ReverseSW_IN"
+		(at 218.44 104.14 0)
+		(effects
+			(font
+				(size 1.27 1.27)
+			)
+			(justify left bottom)
+		)
+	)
+	(label "AcousticWarnSW_IN"
+		(at 229.87 62.23 0)
+		(effects
+			(font
+				(size 1.27 1.27)
+			)
+			(justify left bottom)
+		)
+	)
+	(hierarchical_label "ForwardSW"
 		(shape output)
 		(at 31.75 137.16 180)
@@
 		)
 	)
-	(hierarchical_label "MCU_SW"
+	(hierarchical_label "SpeedLimSW"
 		(shape output)
 		(at 96.52 104.14 180)
@@
 		)
 	)
-	(hierarchical_label "MCU_SW"
+	(hierarchical_label "DirIndSW_L"
 		(shape output)
 		(at 31.75 34.29 180)
@@
 		)
 	)
-	(hierarchical_label "MCU_SW"
+	(hierarchical_label "DirIndSW_R"
 		(shape output)
 		(at 31.75 64.77 180)
@@
 		)
 	)
-	(hierarchical_label "MCU_SW"
+	(hierarchical_label "LightChangeSW"
 		(shape output)
 		(at 173.99 64.77 180)
@@
 		)
 	)
-	(hierarchical_label "MCU_SW"
+	(hierarchical_label "VehicleStartSW"
 		(shape output)
 		(at 30.48 173.99 180)
@@
 		)
 	)
-	(hierarchical_label "MCU_SW"
+	(hierarchical_label "ReverseSW"
 		(shape output)
 		(at 167.64 104.14 180)
@@
 		)
 	)
-	(hierarchical_label "MCU_SW"
+	(hierarchical_label "Assist+SW"
 		(shape output)
 		(at 96.52 137.16 180)
@@
 		)
 	)
-	(hierarchical_label "MCU_SW"
+	(hierarchical_label "MappingSW"
 		(shape output)
 		(at 31.75 104.14 180)
@@
 		)
 	)
-	(hierarchical_label "MCU_SW"
+	(hierarchical_label "Assist-SW"
 		(shape output)
 		(at 167.64 137.16 180)
@@
 		)
 	)
-	(hierarchical_label "MCU_SW"
+	(hierarchical_label "AcousticWarnSW"
 		(shape output)
 		(at 102.87 64.77 180)

Commit message: EMI/EMC meassures implementation + VCU panel interface block
Parts:
- added D22, D46, D47, D48, D49, D50, D51, D52, D53, D54, D55: SMF13A, Diode_SMD:D_SMF, symbol VELION_VCU_Library:SMF13A
- added FB10, FB11, FB12, FB13, FB14, FB4, FB5, FB6, FB7, FB8, FB9: 100R, Inductor_SMD:L_0603_1608Metric, symbol VELION_VCU_Library:FerriteBead_Small
- C87, C88, C89, C90, C91, C92, C93, C96, C97, C98, C99: footprint (none) -> Capacitor_SMD:C_0603_1608Metric; symbol Device:C -> VELION_VCU_Library:C
- D23, D24, D25, D26, D33, D34, D35, D36, D37, D38, D39: footprint PCM_JLCPCB:D_SOD-123 -> Diode_SMD:D_SOD-123; symbol PCM_JLCPCB-Diodes:Switching,1N4148W -> VELION_VCU_Library:Switching,1N4148W
- J18: symbol higo:Z509BM_C_04_00_0000 -> VELION_VCU_Library:Z509BM_C_04_00_0000
- J21: symbol higo:Z809FM_C_04_00_0000 -> VELION_VCU_Library:Z809FM_C_04_00_0000
- R100, R103, R106, R109, R127, R130, R133, R136, R139, R92, R97: footprint PCM_JLCPCB:R_0805 -> Resistor_SMD:R_0805_2012Metric; symbol PCM_JLCPCB-Resistors:0805,1.2kΩ -> VELION_VCU_Library:0805,1.2kΩ
- R101, R104, R107, R110, R128, R131, R134, R137, R94, R95, R98: footprint PCM_JLCPCB:R_0805 -> Resistor_SMD:R_0805_2012Metric; symbol PCM_JLCPCB-Resistors:0805,10kΩ -> VELION_VCU_Library:0805,10kΩ
- R102, R105, R108, R112, R129, R132, R135, R138, R93, R96, R99: footprint PCM_JLCPCB:R_0805 -> Resistor_SMD:R_0805_2012Metric; symbol PCM_JLCPCB-Resistors:0805,33kΩ -> VELION_VCU_Library:0805,33kΩ
Connections:
- net AcousticWarnSW_IN: now also FB5.2; no longer R100.2, R99.1
- net Assist+SW_IN: now also D53.1 (A1), FB10.2; no longer R132.1, R133.2
- net Assist-SW_IN: now also D55.1 (A1), FB14.2; no longer R135.1, R136.2
- net DirIndSW_L_IN: now also FB4.2; no longer R92.2, R93.1
- net DirIndSW_R_IN: now also FB6.2; no longer R96.1, R97.2
- net ForwardSW_IN: now also D52.1 (A1), FB9.2; no longer R129.1, R130.2
- net GND: now also D22.2 (A2), D46.2 (A2), D47.2 (A2), D48.2 (A2), D49.2 (A2), D50.2 (A2), D51.2 (A2), D52.2 (A2), D53.2 (A2), D54.2 (A2), D55.2 (A2)
- net LightChangeSW_IN: now also D48.1 (A1), FB7.2; no longer R102.1, R103.2
- net MappingSW_IN: now also D49.1 (A1), FB11.2; no longer R105.1, R106.2
- net ReverseSW_IN: now also D51.1 (A1), FB13.2; no longer R112.1, R127.2
- net SpeedLimSW_IN: now also D50.1 (A1), FB12.2; no longer R108.1, R109.2
- net VehicleStartSW_IN: now also D54.1 (A1), FB8.2; no longer R138.1, R139.2
- new net: FB12.1, R108.1, R109.2
- new net: D22.1 (A1), FB5.1, R100.2, R99.1
- new net: D47.1 (A1), FB4.1, R92.2, R93.1
- new net: D46.1 (A1), FB6.1, R96.1, R97.2
- new net: FB9.1, R129.1, R130.2
- new net: FB14.1, R135.1, R136.2
- new net: FB7.1, R102.1, R103.2
- new net: FB10.1, R132.1, R133.2
- new net: FB11.1, R105.1, R106.2
- new net: FB13.1, R112.1, R127.2
- new net: FB8.1, R138.1, R139.2
Other:
- moved on the sheet: C90, C93, C98, D26, D35, D38, J21, R101, R102, R103, R110, R112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
