File: InputPower.kicad_sch (KiCad schematic)
At the start: 0 parts

Commit message: DC_DC_blocks + layout
Parts:
- added C133, C134, C151: 10u/25V/X5R, Capacitor_SMD:C_0805_2012Metric, symbol Device:C
- added C135, C136: 22n/X7R, Capacitor_SMD:C_0603_1608Metric, symbol Device:C
- added C137, C138, C149, C153: 100p, Capacitor_SMD:C_0603_1608Metric, symbol Device:C
- added C139, C140, C141, C142, C143, C144: 22u/16V/X7R, Capacitor_SMD:C_0805_2012Metric, symbol Device:C
- added C150, C152: 2n2, Capacitor_SMD:C_0603_1608Metric, symbol Device:C
- added C154: 0u22, Capacitor_SMD:C_0603_1608Metric, symbol Device:C
- added C155: 0u1, Capacitor_SMD:C_0603_1608Metric, symbol Device:C
- added IC3, IC4: RT8293BHZSP, E-M-IntegratedCircuits:SOIC127P600X175-9N, symbol E-M-IntegratedCircuits:RT8293BHZSP
- added L12: 6u8/5A, Inductor_SMD:L_APV_APH0850, symbol Device:L
- added L13: 4u7/5A, Inductor_SMD:L_APV_APH0850, symbol Device:L
- added L15: 1u/5A, Inductor_SMD:L_APV_APH0650, symbol Device:L_Ferrite
- added R144: 62k, Resistor_SMD:R_0603_1608Metric, symbol Device:R
- added R145: 11k8, Resistor_SMD:R_0603_1608Metric, symbol Device:R
- added R146: 75k, Resistor_SMD:R_0603_1608Metric, symbol Device:R
- added R147: 24k, Resistor_SMD:R_0603_1608Metric, symbol Device:R
- added R148, R149: 100k, Resistor_SMD:R_0603_1608Metric, symbol Device:R
- added R150: 33k, Resistor_SMD:R_0603_1608Metric, symbol Device:R
- added R151: 22k, Resistor_SMD:R_0603_1608Metric, symbol Device:R
Connections:
- new net: C154.2, IC4.8 (SS)
- new net: C133.1, C151.1, IC4.2 (VIN), L15.1, R149.1
- new net: C137.2, IC3.5 (FB), R144.2, R145.1
- new net: C136.1, IC3.1 (BOOT)
- new net: C136.2, IC3.3 (SW), L12.1
- new net: C149.2, C150.2, IC3.6 (COMP)
- new net: IC3.7 (EN), R148.2
- new net: C155.2, IC3.8 (SS)
- new net: C135.2, IC4.3 (SW), L13.1
- new net: C138.2, IC4.5 (FB), R146.2, R147.1
- new net: C152.2, C153.2, IC4.6 (COMP)
- new net: C150.1, R150.1
- new net: C152.1, R151.1
- new net: IC4.7 (EN), R149.2
- new net: C135.1, IC4.1 (BOOT)
- new net +12V: C134.1, IC3.2 (VIN), R148.1
- new net +3.3V: C138.1, C140.1, C142.1, C144.1, L13.2, R146.1
- new net +5V: C137.1, C139.1, C141.1, C143.1, L12.2, L15.2, R144.1
- new net GND: C133.2, C134.2, C139.2, C140.2, C141.2, C142.2, C143.2, C144.2, C149.1, C151.2, C153.1, C154.1, C155.1, IC3.4 (GND), IC3.9 (EP), IC4.4 (GND), IC4.9 (EP), R145.2, R147.2, R150.2, R151.2
Other:
- note added: "3A/10W"
- note added: "3A/15W"

Commit message: started pin assignement
Parts:
- renumbered C134 to C1, C135 to C10, C153 to C11, C137 to C12, C138 to C13, C139 to C14, C140 to C15, C141 to C16, C142 to C17, C143 to C18, C144 to C19, C151 to C2, C155 to C3, C133 to C4, C154 to C5, C150 to C6, C136 to C7, C149 to C8, C152 to C9, IC3 to IC1, IC4 to IC2, L15 to L1, L12 to L2, L13 to L3, R148 to R1, R149 to R2, R150 to R3, R151 to R4, R144 to R5, R145 to R6, R146 to R7, R147 to R8
