File: InputPower.kicad_sch (KiCad schematic)
At the start: 32 parts, among them IC3 RT8293BHZSP, IC4 RT8293BHZSP

Commit message: I/O Schematic rebuild from DRAFT by Nathann
Parts:
- added C156: 10u/25V/X5R, Capacitor_SMD:C_0805_2012Metric, symbol Device:C
- added L16: 1u/5A, Inductor_SMD:L_APV_APH0650, symbol Device:L_Ferrite
Connections:
- net +12V: now also L15.2, L16.2; no longer C134.1, IC3.2 (VIN), R148.1
- net +5V: no longer L15.2
- net GND: now also C156.2
- new net: C134.1, C156.1, IC3.2 (VIN), L16.1, R148.1
Other:
- moved on the sheet: C133, C151, L15

Commit message: IMU block implementation
Other:
- moved on the sheet: C133, C134, C135, C136, C137, C138, C139, C140, C141, C142, C143, C144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
