File: InputPower.kicad_sch (KiCad schematic)
At the start: 34 parts, among them IC3 RT8293BHZSP, IC4 RT8293BHZSP

Commit message: EMI/EMC meassures implementation + VCU panel interface block
Parts:
- C133, C134, C135, C136, C137, C138, C139, C140, C141, C142, C143, C144, C149, C150, C151, C152, C153, C154, C155, C156: symbol Device:C -> VELION_VCU_Library:C
- IC3, IC4: symbol E-M-IntegratedCircuits:RT8293BHZSP -> VELION_VCU_Library:RT8293BHZSP
- L12, L13: symbol Device:L -> VELION_VCU_Library:L
- L15, L16: symbol Device:L_Ferrite -> VELION_VCU_Library:L_Ferrite
- R144, R145, R146, R147, R148, R149, R150, R151: symbol Device:R -> VELION_VCU_Library:R
Changed lines of the file:
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@@
 	)
 	(symbol
-		(lib_id "Device:C")
+		(lib_id "VELION_VCU_Library:C")
 		(at 176.53 153.67 180)
 		(unit 1)
@@
 	)
 	(symbol
-		(lib_id "Device:C")
+		(lib_id "VELION_VCU_Library:C")
 		(at 138.43 101.6 0)
 		(unit 1)
@@
 	)
 	(symbol
-		(lib_id "Device:L_Ferrite")
+		(lib_id "VELION_VCU_Library:L_Ferrite")
 		(at 148.59 132.08 180)
 		(unit 1)
@@
 	)
 	(symbol
-		(lib_id "Device:C")
+		(lib_id "VELION_VCU_Library:C")
 		(at 232.41 87.63 0)
 		(unit 1)
@@
 	)
 	(symbol
-		(lib_id "E-M-IntegratedCircuits:RT8293BHZSP")
+		(lib_id "VELION_VCU_Library:RT8293BHZSP")
 		(at 170.18 85.09 0)
 		(unit 1)
@@
 	)
 	(symbol
-		(lib_id "Device:R")
+		(lib_id "VELION_VCU_Library:R")
 		(at 241.3 88.9 0)
 		(unit 1)
@@
 	)
 	(symbol
-		(lib_id "Device:L")
+		(lib_id "VELION_VCU_Library:L")
 		(at 226.06 125.73 90)
 		(unit 1)
@@
 	)
 	(symbol
-		(lib_id "Device:R")
+		(lib_id "VELION_VCU_Library:R")
 		(at 241.3 134.62 0)
 		(unit 1)
@@
 	)
 	(symbol
-		(lib_id "Device:C")
+		(lib_id "VELION_VCU_Library:C")
 		(at 214.63 153.67 270)
 		(unit 1)
@@
 	)
 	(symbol
-		(lib_id "Device:C")
+		(lib_id "VELION_VCU_Library:C")
 		(at 207.01 78.74 90)
 		(unit 1)
@@
 	)
 	(symbol
-		(lib_id "Device:C")
+		(lib_id "VELION_VCU_Library:C")
 		(at 250.19 96.52 0)
 		(unit 1)
@@
 	)
 	(symbol
-		(lib_id "Device:C")
+		(lib_id "VELION_VCU_Library:C")
 		(at 270.51 96.52 0)
 		(unit 1)
@@
 	)
 	(symbol
-		(lib_id "Device:L")
+		(lib_id "VELION_VCU_Library:L")
 		(at 226.06 78.74 90)
 		(unit 1)
@@
 	)
 	(symbol
-		(lib_id "Device:C")
+		(lib_id "VELION_VCU_Library:C")
 		(at 165.1 106.68 180)
 		(unit 1)
@@
 	)
 	(symbol
-		(lib_id "Device:C")
+		(lib_id "VELION_VCU_Library:C")
 		(at 203.2 100.33 270)
 		(unit 1)
@@
 	)
 	(symbol
-		(lib_id "Device:R")
+		(lib_id "VELION_VCU_Library:R")
 		(at 241.3 149.86 0)
 		(unit 1)
@@
 	)
 	(symbol
-		(lib_id "Device:C")
+		(lib_id "VELION_VCU_Library:C")
 		(at 148.59 148.59 0)
 		(unit 1)
@@
 	)
 	(symbol
-		(lib_id "Device:C")
+		(lib_id "VELION_VCU_Library:C")
 		(at 210.82 107.95 270)
 		(unit 1)
@@
 	)
 	(symbol
-		(lib_id "Device:R")
+		(lib_id "VELION_VCU_Library:R")
 		(at 222.25 146.05 90)
 		(unit 1)
@@
 	)
 	(symbol
-		(lib_id "Device:C")
+		(lib_id "VELION_VCU_Library:C")
 		(at 260.35 143.51 0)
 		(unit 1)
@@
 	)
 	(symbol
-		(lib_id "Device:R")
+		(lib_id "VELION_VCU_Library:R")
 		(at 241.3 105.41 0)
 		(unit 1)
@@
 	)
 	(symbol
-		(lib_id "Device:R")
+		(lib_id "VELION_VCU_Library:R")
 		(at 171.45 129.54 0)
 		(unit 1)
@@
 	)
 	(symbol
-		(lib_id "Device:C")
+		(lib_id "VELION_VCU_Library:C")
 		(at 260.35 96.52 0)
 		(unit 1)
@@
 	)
 	(symbol
-		(lib_id "Device:C")
+		(lib_id "VELION_VCU_Library:C")
 		(at 250.19 143.51 0)
 		(unit 1)
@@
 	)
 	(symbol
-		(lib_id "Device:R")
+		(lib_id "VELION_VCU_Library:R")
 		(at 162.56 87.63 0)
 		(unit 1)
@@
 	)
 	(symbol
-		(lib_id "Device:C")
+		(lib_id "VELION_VCU_Library:C")
 		(at 210.82 146.05 270)
 		(unit 1)
@@
 	)
 	(symbol
-		(lib_id "Device:L_Ferrite")
+		(lib_id "VELION_VCU_Library:L_Ferrite")
 		(at 138.43 85.09 180)
 		(unit 1)
@@
 	)
 	(symbol
-		(lib_id "Device:C")
+		(lib_id "VELION_VCU_Library:C")
 		(at 270.51 143.51 0)
 		(unit 1)
@@
 	)
 	(symbol
-		(lib_id "Device:C")
+		(lib_id "VELION_VCU_Library:C")
 		(at 232.41 133.35 0)
 		(unit 1)
@@
 	)
 	(symbol
-		(lib_id "Device:C")
+		(lib_id "VELION_VCU_Library:C")
 		(at 212.09 125.73 90)
 		(unit 1)
@@
 	)
 	(symbol
-		(lib_id "E-M-IntegratedCircuits:RT8293BHZSP")
+		(lib_id "VELION_VCU_Library:RT8293BHZSP")
 		(at 179.07 130.81 0)
 		(unit 1)
@@
 	)
 	(symbol
-		(lib_id "Device:C")
+		(lib_id "VELION_VCU_Library:C")
 		(at 153.67 101.6 0)
 		(unit 1)
@@
 	)
 	(symbol
-		(lib_id "Device:C")
+		(lib_id "VELION_VCU_Library:C")
 		(at 160.02 148.59 0)
 		(unit 1)
@@
 	)
 	(symbol
-		(lib_id "Device:R")
+		(lib_id "VELION_VCU_Library:R")
 		(at 219.71 100.33 90)
 		(unit 1)
