File: PowertrainInterface.kicad_sch (KiCad schematic)
At the start: 15 parts, among them J7 IEC61076-2_M8_B-coding_01x03_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, U4 CA-IS2062W

Commit message: started pin assignement
Parts:
- renumbered C19 to C74, C18 to C75, C17 to C76, C16 to C77, C15 to C78, C20 to C79, D5 to D15, J7 to J25, L3 to L5, R8 to R66, R9 to R67, R11 to R68, R12 to R69, R10 to R70, U4 to U17
Changed lines of the file:
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@@
 		(dnp no)
 		(fields_autoplaced yes)
-		(property "Reference" "#PWR058"
+		(property "Reference" "#PWR0179"
 			(at 64.77 58.42 0)
 			(hide yes)
@@
 			(project "MainBoard"
 				(path "/6deb7572-40fc-4be3-9f80-b7a356c09b38/d8a37f98-2a8b-4436-b9d3-44ea6584471e"
-					(reference "#PWR058")
+					(reference "#PWR0179")
 					(unit 1)
 				)
@@
 		(in_pos_files yes)
 		(dnp no)
-		(property "Reference" "C15"
+		(property "Reference" "C78"
 			(at 165.608 54.864 90)
 			(show_name no)
@@
 			(project "MainBoard"
 				(path "/6deb7572-40fc-4be3-9f80-b7a356c09b38/d8a37f98-2a8b-4436-b9d3-44ea6584471e"
-					(reference "C15")
+					(reference "C78")
 					(unit 1)
 				)
@@
 		(dnp no)
 		(fields_autoplaced yes)
-		(property "Reference" "L3"
+		(property "Reference" "L5"
 			(at 74.93 52.07 90)
 			(show_name no)
@@
 			(project "MainBoard"
 				(path "/6deb7572-40fc-4be3-9f80-b7a356c09b38/d8a37f98-2a8b-4436-b9d3-44ea6584471e"
-					(reference "L3")
+					(reference "L5")
 					(unit 1)
 				)
@@
 		(dnp no)
 		(fields_autoplaced yes)
-		(property "Reference" "#PWR070"
+		(property "Reference" "#PWR0190"
 			(at 175.26 95.25 0)
 			(hide yes)
@@
 			(project "MainBoard"
 				(path "/6deb7572-40fc-4be3-9f80-b7a356c09b38/d8a37f98-2a8b-4436-b9d3-44ea6584471e"
-					(reference "#PWR070")
+					(reference "#PWR0190")
 					(unit 1)
 				)
@@
 		(dnp no)
 		(fields_autoplaced yes)
-		(property "Reference" "#PWR068"
+		(property "Reference" "#PWR0188"
 			(at 171.45 52.07 0)
 			(hide yes)
@@
 			(project "MainBoard"
 				(path "/6deb7572-40fc-4be3-9f80-b7a356c09b38/d8a37f98-2a8b-4436-b9d3-44ea6584471e"
-					(reference "#PWR068")
+					(reference "#PWR0188")
 					(unit 1)
 				)
@@
 		(dnp no)
 		(fields_autoplaced yes)
-		(property "Reference" "#PWR065"
+		(property "Reference" "#PWR0185"
 			(at 153.67 100.33 0)
 			(hide yes)
@@
 			(project "MainBoard"
 				(path "/6deb7572-40fc-4be3-9f80-b7a356c09b38/d8a37f98-2a8b-4436-b9d3-44ea6584471e"
-					(reference "#PWR065")
+					(reference "#PWR0185")
 					(unit 1)
 				)
@@
 		(in_pos_files yes)
 		(dnp no)
-		(property "Reference" "C19"
+		(property "Reference" "C74"
 			(at 62.23 75.946 90)
 			(show_name no)
@@
 			(project "MainBoard"
 				(path "/6deb7572-40fc-4be3-9f80-b7a356c09b38/d8a37f98-2a8b-4436-b9d3-44ea6584471e"
-					(reference "C19")
+					(reference "C74")
 					(unit 1)
 				)
@@
 		(in_pos_files yes)
 		(dnp no)
-		(property "Reference" "C18"
+		(property "Reference" "C75"
 			(at 81.28 75.946 90)
 			(show_name no)
@@
 			(project "MainBoard"
 				(path "/6deb7572-40fc-4be3-9f80-b7a356c09b38/d8a37f98-2a8b-4436-b9d3-44ea6584471e"
-					(reference "C18")
+					(reference "C75")
 					(unit 1)
 				)
@@
 		(dnp no)
 		(fields_autoplaced yes)
-		(property "Reference" "#PWR063"
+		(property "Reference" "#PWR0184"
 			(at 114.3 72.39 0)
 			(hide yes)
@@
 			(project "MainBoard"
 				(path "/6deb7572-40fc-4be3-9f80-b7a356c09b38/d8a37f98-2a8b-4436-b9d3-44ea6584471e"
-					(reference "#PWR063")
+					(reference "#PWR0184")
 					(unit 1)
 				)
@@
 		(dnp no)
 		(fields_autoplaced yes)
-		(property "Reference" "#PWR059"
+		(property "Reference" "#PWR0180"
 			(at 64.77 82.55 0)
 			(hide yes)
@@
 			(project "MainBoard"
 				(path "/6deb7572-40fc-4be3-9f80-b7a356c09b38/d8a37f98-2a8b-4436-b9d3-44ea6584471e"
-					(reference "#PWR059")
+					(reference "#PWR0180")
 					(unit 1)
 				)
@@
 		(in_pos_files yes)
 		(dnp no)
-		(property "Reference" "R9"
+		(property "Reference" "R67"
 			(at 172.212 82.55 90)
 			(show_name no)
@@
 			(project "MainBoard"
 				(path "/6deb7572-40fc-4be3-9f80-b7a356c09b38/d8a37f98-2a8b-4436-b9d3-44ea6584471e"
-					(reference "R9")
+					(reference "R67")
 					(unit 1)
 				)
@@
 		(dnp no)
 		(fields_autoplaced yes)
-		(property "Reference" "#PWR067"
+		(property "Reference" "#PWR0187"
 			(at 171.45 41.91 0)
 			(hide yes)
@@
 			(project "MainBoard"
 				(path "/6deb7572-40fc-4be3-9f80-b7a356c09b38/d8a37f98-2a8b-4436-b9d3-44ea6584471e"
-					(reference "#PWR067")
+					(reference "#PWR0187")
 					(unit 1)
 				)
@@
 		(in_pos_files yes)
 		(dnp no)
-		(property "Reference" "C16"
+		(property "Reference" "C77"
 			(at 165.862 44.704 90)
 			(show_name no)
@@
 			(project "MainBoard"
 				(path "/6deb7572-40fc-4be3-9f80-b7a356c09b38/d8a37f98-2a8b-4436-b9d3-44ea6584471e"
-					(reference "C16")
+					(reference "C77")
 					(unit 1)
 				)
@@
 		(dnp no)
 		(fields_autoplaced yes)
-		(property "Reference" "#PWR071"
+		(property "Reference" "#PWR0191"
 			(at 207.01 125.73 0)
 			(hide yes)
@@
 			(project "MainBoard"
 				(path "/6deb7572-40fc-4be3-9f80-b7a356c09b38/d8a37f98-2a8b-4436-b9d3-44ea6584471e"
-					(reference "#PWR071")
+					(reference "#PWR0191")
 					(unit 1)
 				)
@@
 		(dnp no)
 		(fields_autoplaced yes)
-		(property "Reference" "#PWR062"
+		(property "Reference" "#PWR0183"
 			(at 113.03 99.06 0)
 			(hide yes)
@@
 			(project "MainBoard"
 				(path "/6deb7572-40fc-4be3-9f80-b7a356c09b38/d8a37f98-2a8b-4436-b9d3-44ea6584471e"
-					(reference "#PWR062")
+					(reference "#PWR0183")
 					(unit 1)
 				)
@@
 		(in_pos_files yes)
 		(dnp no)
-		(property "Reference" "D5"
+		(property "Reference" "D15"
 			(at 183.134 81.534 0)
 			(show_name no)
@@
 			(project "MainBoard"
 				(path "/6deb7572-40fc-4be3-9f80-b7a356c09b38/d8a37f98-2a8b-4436-b9d3-44ea6584471e"
-					(reference "D5")
+					(reference "D15")
 					(unit 1)
 				)
@@
 		(in_pos_files yes)
 		(dnp no)
-		(property "Reference" "R10"
+		(property "Reference" "R70"
 			(at 212.344 96.52 90)
 			(show_name no)
@@
 			(project "MainBoard"
 				(path "/6deb7572-40fc-4be3-9f80-b7a356c09b38/d8a37f98-2a8b-4436-b9d3-44ea6584471e"
-					(reference "R10")
+					(reference "R70")
 					(unit 1)
 				)
@@
 		(dnp no)
 		(fields_autoplaced yes)
-		(property "Reference" "#PWR060"
+		(property "Reference" "#PWR0181"
 			(at 83.82 82.55 0)
 			(hide yes)
@@
 			(project "MainBoard"
 				(path "/6deb7572-40fc-4be3-9f80-b7a356c09b38/d8a37f98-2a8b-4436-b9d3-44ea6584471e"
-					(reference "#PWR060")
+					(reference "#PWR0181")
 					(unit 1)
 				)
@@
 		(dnp no)
 		(fields_autoplaced yes)
-		(property "Reference" "#PWR066"
+		(property "Reference" "#PWR0186"
 			(at 158.75 73.66 0)
 			(hide yes)
@@
 			(project "MainBoard"
 				(path "/6deb7572-40fc-4be3-9f80-b7a356c09b38/d8a37f98-2a8b-4436-b9d3-44ea6584471e"
-					(reference "#PWR066")
+					(reference "#PWR0186")
 					(unit 1)
 				)
@@
 		(in_pos_files yes)
 		(dnp no)
-		(property "Reference" "C20"
+		(property "Reference" "C79"
 			(at 211.074 104.902 90)
 			(show_name no)
@@
 			(project "MainBoard"
 				(path "/6deb7572-40fc-4be3-9f80-b7a356c09b38/d8a37f98-2a8b-4436-b9d3-44ea6584471e"
-					(reference "C20")
+					(reference "C79")
 					(unit 1)
 				)
@@
 		(in_pos_files yes)
 		(dnp no)
-		(property "Reference" "J7"
+		(property "Reference" "J25"
 			(at 216.662 74.676 0)
 			(show_name no)
@@
 			(project "MainBoard"
 				(path "/6deb7572-40fc-4be3-9f80-b7a356c09b38/d8a37f98-2a8b-4436-b9d3-44ea6584471e"
-					(reference "J7")
+					(reference "J25")
 					(unit 1)
 				)
@@
 		(dnp no)
 		(fields_autoplaced yes)
-		(property "Reference" "#PWR061"
+		(property "Reference" "#PWR0182"
 			(at 96.52 82.55 0)
 			(hide yes)
@@
 			(project "MainBoard"
 				(path "/6deb7572-40fc-4be3-9f80-b7a356c09b38/d8a37f98-2a8b-4436-b9d3-44ea6584471e"
-					(reference "#PWR061")
+					(reference "#PWR0182")
 					(unit 1)
 				)
@@
 		(in_pos_files yes)
 		(dnp no)
-		(property "Reference" "C17"
+		(property "Reference" "C76"
 			(at 94.234 75.438 90)
 			(show_name no)
@@
 			(project "MainBoard"
 				(path "/6deb7572-40fc-4be3-9f80-b7a356c09b38/d8a37f98-2a8b-4436-b9d3-44ea6584471e"
-					(reference "C17")
+					(reference "C76")
 					(unit 1)
 				)
@@
 		(in_pos_files yes)
 		(dnp no)
-		(property "Reference" "R8"
+		(property "Reference" "R66"
 			(at 172.212 64.77 90)
 			(show_name no)
@@
 			(project "MainBoard"
 				(path "/6deb7572-40fc-4be3-9f80-b7a356c09b38/d8a37f98-2a8b-4436-b9d3-44ea6584471e"
-					(reference "R8")
+					(reference "R66")
 					(unit 1)
 				)
@@
 		(in_pos_files yes)
 		(dnp no)
-		(property "Reference" "R11"
+		(property "Reference" "R68"
 			(at 184.912 55.88 90)
 			(show_name no)
@@
 			(project "MainBoard"
 				(path "/6deb7572-40fc-4be3-9f80-b7a356c09b38/d8a37f98-2a8b-4436-b9d3-44ea6584471e"
-					(reference "R11")
+					(reference "R68")
 					(unit 1)
 				)
@@
 		(dnp no)
 		(fields_autoplaced yes)
-		(property "Reference" "U4"
+		(property "Reference" "U17"
 			(at 133.35 50.8 0)
 			(show_name no)
@@
 			(project "MainBoard"
 				(path "/6deb7572-40fc-4be3-9f80-b7a356c09b38/d8a37f98-2a8b-4436-b9d3-44ea6584471e"
-					(reference "U4")
+					(reference "U17")
 					(unit 1)
 				)
@@
 		(dnp no)
 		(fields_autoplaced yes)
-		(property "Reference" "#PWR069"
+		(property "Reference" "#PWR0189"
 			(at 173.99 76.2 0)
 			(hide yes)
@@
 			(project "MainBoard"
 				(path "/6deb7572-40fc-4be3-9f80-b7a356c09b38/d8a37f98-2a8b-4436-b9d3-44ea6584471e"
-					(reference "#PWR069")
+					(reference "#PWR0189")
 					(unit 1)
 				)
@@
 		(in_pos_files yes)
 		(dnp no)
-		(property "Reference" "R12"
+		(property "Reference" "R69"
 			(at 187.452 92.71 90)
 			(show_name no)
@@
 			(project "MainBoard"
 				(path "/6deb7572-40fc-4be3-9f80-b7a356c09b38/d8a37f98-2a8b-4436-b9d3-44ea6584471e"
-					(reference "R12")
-					(unit 1)
-				)
+					(reference "R69")
+					(unit 1)
+				)
