File: USB_PD.kicad_sch (KiCad schematic)
At the start: 29 parts, among them IC2 STUSB4500LQTR, J15 USB_C_2.0, Q6 STL9P3LLH6, Q7 STL9P3LLH6, U27 USBLC6-2P6

Commit message: added output driver
Parts:
- renumbered C112 to C114, C111 to C115, C110 to C116, C109 to C117, C108 to C118, C113 to C119, D28 to D31, D29 to D32, D27 to D33, D30 to D34, IC2 to IC5, J15 to J24, Q6 to Q8, Q7 to Q9, R111 to R112, R119 to R126, R120 to R127, R116 to R128, R117 to R129, R121 to R130, R122 to R131, R123 to R132, R118 to R133, R125 to R134, R124 to R135, TP11 to TP15, TP22 to TP24, TP23 to TP25, U27 to U28

Commit message: started pin assignement
Parts:
- renumbered C114 to C62, C115 to C63, C116 to C64, C117 to C65, C118 to C66, C119 to C67, D34 to D10, D31 to D7, D32 to D8, D33 to D9, IC5 to IC3, J24 to J23, Q8 to Q1, Q9 to Q2, R112 to R44, R126 to R45, R127 to R46, R128 to R47, R129 to R48, R130 to R49, R131 to R50, R132 to R51, R133 to R52, R134 to R53, R135 to R54, TP15 to TP6, TP24 to TP7, TP25 to TP8, U28 to U15
