File: USB_PD.kicad_sch (KiCad schematic)
At the start: 29 parts, among them IC2 STUSB4500LQTR, J15 USB_C_2.0, Q6 STL9P3LLH6, Q7 STL9P3LLH6, U27 USBLC6-2P6

Commit message: EMI/EMC meassures implementation + VCU panel interface block
Parts:
- C108, C109, C110, C111, C112, C113: symbol Device:C -> VELION_VCU_Library:C
- D27: symbol Device:D_Schottky -> VELION_VCU_Library:D_Schottky
- D28: symbol Device:D_Dual_CommonAnode_KKA_Split -> VELION_VCU_Library:D_Dual_CommonAnode_KKA_Split
- D29, D30: symbol Diode:SMAJ28A -> VELION_VCU_Library:SMAJ28A
- IC2: symbol E-M-IntegratedCircuits:STUSB4500LQTR -> VELION_VCU_Library:STUSB4500LQTR
- J15: symbol Connector:USB_C_Receptacle_USB2.0 -> VELION_VCU_Library:USB_C_Receptacle_USB2.0
- Q6, Q7: symbol Transistor_FET:DMP3013SFV -> VELION_VCU_Library:DMP3013SFV
- R111: symbol CD-ACSCREEN-1-eagle-import:rcl_R-EU_R0402 -> VELION_VCU_Library:rcl_R-EU_R0402
- R116, R117, R118, R119, R120, R121, R122, R123, R124, R125: symbol Device:R -> VELION_VCU_Library:R
- TP11, TP22, TP23: symbol Connector:TestPoint -> VELION_VCU_Library:TestPoint
- U27: symbol Power_Protection:USBLC6-2P6 -> VELION_VCU_Library:USBLC6-2P6
Changed lines of the file:
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@@
 	)
 	(symbol
-		(lib_id "Device:D_Dual_CommonAnode_KKA_Split")
+		(lib_id "VELION_VCU_Library:D_Dual_CommonAnode_KKA_Split")
 		(at 82.55 130.81 90)
 		(unit 2)
@@
 	)
 	(symbol
-		(lib_id "Device:R")
+		(lib_id "VELION_VCU_Library:R")
 		(at 191.77 120.65 0)
 		(unit 1)
@@
 	)
 	(symbol
-		(lib_id "Device:R")
+		(lib_id "VELION_VCU_Library:R")
 		(at 187.96 106.68 90)
 		(unit 1)
@@
 	)
 	(symbol
-		(lib_id "Device:R")
+		(lib_id "VELION_VCU_Library:R")
 		(at 113.03 82.55 0)
 		(unit 1)
@@
 	)
 	(symbol
-		(lib_id "CD-ACSCREEN-1-eagle-import:rcl_R-EU_R0402")
+		(lib_id "VELION_VCU_Library:rcl_R-EU_R0402")
 		(at 22.86 80.01 270)
 		(mirror x)
@@
 	)
 	(symbol
-		(lib_id "Connector:TestPoint")
+		(lib_id "VELION_VCU_Library:TestPoint")
 		(at 256.54 147.32 270)
 		(unit 1)
@@
 	)
 	(symbol
-		(lib_id "Device:C")
+		(lib_id "VELION_VCU_Library:C")
 		(at 78.74 95.25 0)
 		(unit 1)
@@
 	)
 	(symbol
-		(lib_id "Connector:TestPoint")
+		(lib_id "VELION_VCU_Library:TestPoint")
 		(at 256.54 154.94 270)
 		(unit 1)
@@
 	)
 	(symbol
-		(lib_id "Transistor_FET:DMP3013SFV")
+		(lib_id "VELION_VCU_Library:DMP3013SFV")
 		(at 180.34 29.21 270)
 		(mirror x)
@@
 	)
 	(symbol
-		(lib_id "Connector:USB_C_Receptacle_USB2.0")
+		(lib_id "VELION_VCU_Library:USB_C_Receptacle_USB2.0")
 		(at 30.48 41.91 0)
 		(unit 1)
@@
 	)
 	(symbol
-		(lib_id "Transistor_FET:DMP3013SFV")
+		(lib_id "VELION_VCU_Library:DMP3013SFV")
 		(at 214.63 29.21 90)
 		(unit 1)
@@
 	)
 	(symbol
-		(lib_id "Device:R")
+		(lib_id "VELION_VCU_Library:R")
 		(at 162.56 66.04 0)
 		(unit 1)
@@
 	)
 	(symbol
-		(lib_id "Connector:TestPoint")
+		(lib_id "VELION_VCU_Library:TestPoint")
 		(at 146.05 22.86 0)
 		(unit 1)
@@
 	)
 	(symbol
-		(lib_id "Device:C")
+		(lib_id "VELION_VCU_Library:C")
 		(at 107.95 148.59 0)
 		(unit 1)
@@
 	)
 	(symbol
-		(lib_id "Device:C")
+		(lib_id "VELION_VCU_Library:C")
 		(at 99.06 96.52 0)
 		(unit 1)
@@
 	)
 	(symbol
-		(lib_id "Power_Protection:USBLC6-2P6")
+		(lib_id "VELION_VCU_Library:USBLC6-2P6")
 		(at 99.06 52.07 90)
 		(unit 1)
@@
 	)
 	(symbol
-		(lib_id "Device:C")
+		(lib_id "VELION_VCU_Library:C")
 		(at 99.06 148.59 0)
 		(unit 1)
@@
 	)
 	(symbol
-		(lib_id "Device:D_Dual_CommonAnode_KKA_Split")
+		(lib_id "VELION_VCU_Library:D_Dual_CommonAnode_KKA_Split")
 		(at 72.39 130.81 90)
 		(unit 1)
@@
 	)
 	(symbol
-		(lib_id "Device:R")
+		(lib_id "VELION_VCU_Library:R")
 		(at 128.27 153.67 0)
 		(unit 1)
@@
 	)
 	(symbol
-		(lib_id "Diode:SMAJ28A")
+		(lib_id "VELION_VCU_Library:SMAJ28A")
 		(at 271.78 64.77 270)
 		(unit 1)
@@
 	)
 	(symbol
-		(lib_id "Device:R")
+		(lib_id "VELION_VCU_Library:R")
 		(at 172.72 55.88 90)
 		(unit 1)
@@
 	)
 	(symbol
-		(lib_id "E-M-IntegratedCircuits:STUSB4500LQTR")
+		(lib_id "VELION_VCU_Library:STUSB4500LQTR")
 		(at 143.51 101.6 0)
 		(unit 1)
@@
 	)
 	(symbol
-		(lib_id "Device:D_Schottky")
+		(lib_id "VELION_VCU_Library:D_Schottky")
 		(at 99.06 82.55 90)
 		(unit 1)
@@
 	)
 	(symbol
-		(lib_id "Device:C")
+		(lib_id "VELION_VCU_Library:C")
 		(at 190.5 41.91 0)
 		(unit 1)
@@
 	)
 	(symbol
-		(lib_id "Device:R")
+		(lib_id "VELION_VCU_Library:R")
 		(at 182.88 147.32 0)
 		(unit 1)
@@
 	)
 	(symbol
-		(lib_id "Diode:SMAJ28A")
+		(lib_id "VELION_VCU_Library:SMAJ28A")
 		(at 88.9 93.98 270)
 		(unit 1)
@@
 	)
 	(symbol
-		(lib_id "Device:R")
+		(lib_id "VELION_VCU_Library:R")
 		(at 113.03 99.06 0)
 		(unit 1)
@@
 	)
 	(symbol
-		(lib_id "Device:R")
+		(lib_id "VELION_VCU_Library:R")
 		(at 137.16 153.67 0)
 		(unit 1)
@@
 	)
 	(symbol
-		(lib_id "Device:R")
+		(lib_id "VELION_VCU_Library:R")
 		(at 162.56 45.72 0)
 		(unit 1)
@@
 	)
 	(symbol
-		(lib_id "Device:C")
+		(lib_id "VELION_VCU_Library:C")
 		(at 118.11 148.59 0)
 		(unit 1)
