File: inputAnalog.kicad_sch (KiCad schematic)
At the start: 4 parts

Commit message: wiring MCU to input and ouput
Changed lines of the file:
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@@
 	)
 	(hierarchical_label "MCU_AN"
-		(shape input)
+		(shape output)
 		(at 137.16 95.25 0)
 		(effects
@@
 		(instances
 			(project "MainBoard"
+				(path "/6deb7572-40fc-4be3-9f80-b7a356c09b38/0c155571-1bd8-4bec-bb4f-8e0bfac8183f"
+					(reference "D25")
+					(unit 1)
+				)
+				(path "/6deb7572-40fc-4be3-9f80-b7a356c09b38/316d4f3f-7ca7-4a40-9e18-39726f76d5ff"
+					(reference "D36")
+					(unit 1)
+				)
 				(path "/6deb7572-40fc-4be3-9f80-b7a356c09b38/3d38696f-347d-4199-9e08-23c1c8c9195d"
 					(reference "D6")
+					(unit 1)
+				)
+				(path "/6deb7572-40fc-4be3-9f80-b7a356c09b38/4bb5f3ae-ce82-4338-998d-62be1b297bde"
+					(reference "D22")
+					(unit 1)
+				)
+				(path "/6deb7572-40fc-4be3-9f80-b7a356c09b38/de4c83ca-265a-403e-acdd-e77774d3be85"
+					(reference "D39")
 					(unit 1)
 				)
@@
 		(instances
 			(project "MainBoard"
+				(path "/6deb7572-40fc-4be3-9f80-b7a356c09b38/0c155571-1bd8-4bec-bb4f-8e0bfac8183f"
+					(reference "C40")
+					(unit 1)
+				)
+				(path "/6deb7572-40fc-4be3-9f80-b7a356c09b38/316d4f3f-7ca7-4a40-9e18-39726f76d5ff"
+					(reference "C43")
+					(unit 1)
+				)
 				(path "/6deb7572-40fc-4be3-9f80-b7a356c09b38/3d38696f-347d-4199-9e08-23c1c8c9195d"
 					(reference "C3")
+					(unit 1)
+				)
+				(path "/6deb7572-40fc-4be3-9f80-b7a356c09b38/4bb5f3ae-ce82-4338-998d-62be1b297bde"
+					(reference "C37")
+					(unit 1)
+				)
+				(path "/6deb7572-40fc-4be3-9f80-b7a356c09b38/de4c83ca-265a-403e-acdd-e77774d3be85"
+					(reference "C46")
 					(unit 1)
 				)
@@
 		(instances
 			(project "MainBoard"
+				(path "/6deb7572-40fc-4be3-9f80-b7a356c09b38/0c155571-1bd8-4bec-bb4f-8e0bfac8183f"
+					(reference "R77")
+					(unit 1)
+				)
+				(path "/6deb7572-40fc-4be3-9f80-b7a356c09b38/316d4f3f-7ca7-4a40-9e18-39726f76d5ff"
+					(reference "R85")
+					(unit 1)
+				)
 				(path "/6deb7572-40fc-4be3-9f80-b7a356c09b38/3d38696f-347d-4199-9e08-23c1c8c9195d"
 					(reference "R13")
+					(unit 1)
+				)
+				(path "/6deb7572-40fc-4be3-9f80-b7a356c09b38/4bb5f3ae-ce82-4338-998d-62be1b297bde"
+					(reference "R69")
+					(unit 1)
+				)
+				(path "/6deb7572-40fc-4be3-9f80-b7a356c09b38/de4c83ca-265a-403e-acdd-e77774d3be85"
+					(reference "R93")
 					(unit 1)
 				)
@@
 		(instances
 			(project "MainBoard"
+				(path "/6deb7572-40fc-4be3-9f80-b7a356c09b38/0c155571-1bd8-4bec-bb4f-8e0bfac8183f"
+					(reference "#PWR0240")
+					(unit 1)
+				)
+				(path "/6deb7572-40fc-4be3-9f80-b7a356c09b38/316d4f3f-7ca7-4a40-9e18-39726f76d5ff"
+					(reference "#PWR0250")
+					(unit 1)
+				)
 				(path "/6deb7572-40fc-4be3-9f80-b7a356c09b38/3d38696f-347d-4199-9e08-23c1c8c9195d"
 					(reference "#PWR0150")
+					(unit 1)
+				)
+				(path "/6deb7572-40fc-4be3-9f80-b7a356c09b38/4bb5f3ae-ce82-4338-998d-62be1b297bde"
+					(reference "#PWR0224")
+					(unit 1)
+				)
+				(path "/6deb7572-40fc-4be3-9f80-b7a356c09b38/de4c83ca-265a-403e-acdd-e77774d3be85"
+					(reference "#PWR0258")
 					(unit 1)
 				)
@@
 		(instances
 			(project "MainBoard"
+				(path "/6deb7572-40fc-4be3-9f80-b7a356c09b38/0c155571-1bd8-4bec-bb4f-8e0bfac8183f"
+					(reference "R78")
+					(unit 1)
+				)
+				(path "/6deb7572-40fc-4be3-9f80-b7a356c09b38/316d4f3f-7ca7-4a40-9e18-39726f76d5ff"
+					(reference "R86")
+					(unit 1)
+				)
 				(path "/6deb7572-40fc-4be3-9f80-b7a356c09b38/3d38696f-347d-4199-9e08-23c1c8c9195d"
 					(reference "R14")
+					(unit 1)
+				)
+				(path "/6deb7572-40fc-4be3-9f80-b7a356c09b38/4bb5f3ae-ce82-4338-998d-62be1b297bde"
+					(reference "R70")
+					(unit 1)
+				)
+				(path "/6deb7572-40fc-4be3-9f80-b7a356c09b38/de4c83ca-265a-403e-acdd-e77774d3be85"
+					(reference "R94")
 					(unit 1)
 				)
@@
 		(instances
 			(project "MainBoard"
+				(path "/6deb7572-40fc-4be3-9f80-b7a356c09b38/0c155571-1bd8-4bec-bb4f-8e0bfac8183f"
+					(reference "#PWR0239")
+					(unit 1)
+				)
+				(path "/6deb7572-40fc-4be3-9f80-b7a356c09b38/316d4f3f-7ca7-4a40-9e18-39726f76d5ff"
+					(reference "#PWR0249")
+					(unit 1)
+				)
 				(path "/6deb7572-40fc-4be3-9f80-b7a356c09b38/3d38696f-347d-4199-9e08-23c1c8c9195d"
 					(reference "#PWR0149")
 					(unit 1)
 				)
+				(path "/6deb7572-40fc-4be3-9f80-b7a356c09b38/4bb5f3ae-ce82-4338-998d-62be1b297bde"
+					(reference "#PWR0223")
+					(unit 1)
+				)
+				(path "/6deb7572-40fc-4be3-9f80-b7a356c09b38/de4c83ca-265a-403e-acdd-e77774d3be85"
+					(reference "#PWR0257")
+					(unit 1)
+				)

Commit message: started pin assignement
Parts:
- removed R13: 10k, symbol Device:R
- removed R14: 15k, symbol Device:R
- added R33: 10kΩ, PCM_JLCPCB:R_0805, symbol PCM_JLCPCB-Resistors:0805,10kΩ
- added R34: 15kΩ, PCM_JLCPCB:R_0805, symbol PCM_JLCPCB-Resistors:0805,15kΩ
- renumbered C3 to C58, D6 to D3
Connections:
- net AN: now also R33.1
- net GND: now also R34.2
- net MCU_AN: now also R33.2, R34.1
