File: inputPAS.kicad_sch (KiCad schematic)
At the start: 10 parts

Commit message: wiring MCU to input and ouput
Changed lines of the file:
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@@
 	)
 	(hierarchical_label "MCU_PAS_A"
-		(shape input)
+		(shape output)
 		(at 120.65 95.25 0)
 		(effects
@@
 	)
 	(hierarchical_label "MCU_PAS_B"
-		(shape input)
+		(shape output)
 		(at 120.65 146.05 0)
 		(effects
@@
 					(unit 1)
 				)
+				(path "/6deb7572-40fc-4be3-9f80-b7a356c09b38/8c1e6824-86fa-49c6-92ab-5b5974896eb4"
+					(reference "R90")
+					(unit 1)
+				)
+				(path "/6deb7572-40fc-4be3-9f80-b7a356c09b38/97176d4a-f469-4b3e-946d-de72b475fa7f"
+					(reference "R82")
+					(unit 1)
+				)
+				(path "/6deb7572-40fc-4be3-9f80-b7a356c09b38/bb90eeae-f6b7-4ab0-91ca-1f494e8dc0e5"
+					(reference "R74")
+					(unit 1)
+				)
 			)
 		)
@@
 					(unit 1)
 				)
+				(path "/6deb7572-40fc-4be3-9f80-b7a356c09b38/8c1e6824-86fa-49c6-92ab-5b5974896eb4"
+					(reference "#PWR0252")
+					(unit 1)
+				)
+				(path "/6deb7572-40fc-4be3-9f80-b7a356c09b38/97176d4a-f469-4b3e-946d-de72b475fa7f"
+					(reference "#PWR0244")
+					(unit 1)
+				)
+				(path "/6deb7572-40fc-4be3-9f80-b7a356c09b38/bb90eeae-f6b7-4ab0-91ca-1f494e8dc0e5"
+					(reference "#PWR0226")
+					(unit 1)
+				)
 			)
 		)
@@
 					(unit 1)
 				)
+				(path "/6deb7572-40fc-4be3-9f80-b7a356c09b38/8c1e6824-86fa-49c6-92ab-5b5974896eb4"
+					(reference "#PWR0251")
+					(unit 1)
+				)
+				(path "/6deb7572-40fc-4be3-9f80-b7a356c09b38/97176d4a-f469-4b3e-946d-de72b475fa7f"
+					(reference "#PWR0243")
+					(unit 1)
+				)
+				(path "/6deb7572-40fc-4be3-9f80-b7a356c09b38/bb90eeae-f6b7-4ab0-91ca-1f494e8dc0e5"
+					(reference "#PWR0225")
+					(unit 1)
+				)
 			)
 		)
@@
 					(unit 1)
 				)
+				(path "/6deb7572-40fc-4be3-9f80-b7a356c09b38/8c1e6824-86fa-49c6-92ab-5b5974896eb4"
+					(reference "D38")
+					(unit 1)
+				)
+				(path "/6deb7572-40fc-4be3-9f80-b7a356c09b38/97176d4a-f469-4b3e-946d-de72b475fa7f"
+					(reference "D35")
+					(unit 1)
+				)
+				(path "/6deb7572-40fc-4be3-9f80-b7a356c09b38/bb90eeae-f6b7-4ab0-91ca-1f494e8dc0e5"
+					(reference "D24")
+					(unit 1)
+				)
 			)
 		)
@@
 					(unit 1)
 				)
+				(path "/6deb7572-40fc-4be3-9f80-b7a356c09b38/8c1e6824-86fa-49c6-92ab-5b5974896eb4"
+					(reference "R88")
+					(unit 1)
+				)
+				(path "/6deb7572-40fc-4be3-9f80-b7a356c09b38/97176d4a-f469-4b3e-946d-de72b475fa7f"
+					(reference "R80")
+					(unit 1)
+				)
+				(path "/6deb7572-40fc-4be3-9f80-b7a356c09b38/bb90eeae-f6b7-4ab0-91ca-1f494e8dc0e5"
+					(reference "R72")
+					(unit 1)
+				)
 			)
 		)
@@
 					(unit 1)
 				)
+				(path "/6deb7572-40fc-4be3-9f80-b7a356c09b38/8c1e6824-86fa-49c6-92ab-5b5974896eb4"
+					(reference "R91")
+					(unit 1)
+				)
+				(path "/6deb7572-40fc-4be3-9f80-b7a356c09b38/97176d4a-f469-4b3e-946d-de72b475fa7f"
+					(reference "R83")
+					(unit 1)
+				)
+				(path "/6deb7572-40fc-4be3-9f80-b7a356c09b38/bb90eeae-f6b7-4ab0-91ca-1f494e8dc0e5"
+					(reference "R75")
+					(unit 1)
+				)
 			)
 		)
@@
 					(unit 1)
 				)
+				(path "/6deb7572-40fc-4be3-9f80-b7a356c09b38/8c1e6824-86fa-49c6-92ab-5b5974896eb4"
+					(reference "R89")
+					(unit 1)
+				)
+				(path "/6deb7572-40fc-4be3-9f80-b7a356c09b38/97176d4a-f469-4b3e-946d-de72b475fa7f"
+					(reference "R81")
+					(unit 1)
+				)
+				(path "/6deb7572-40fc-4be3-9f80-b7a356c09b38/bb90eeae-f6b7-4ab0-91ca-1f494e8dc0e5"
+					(reference "R73")
+					(unit 1)
+				)
 			)
 		)
@@
 					(unit 1)
 				)
+				(path "/6deb7572-40fc-4be3-9f80-b7a356c09b38/8c1e6824-86fa-49c6-92ab-5b5974896eb4"
+					(reference "#PWR0256")
+					(unit 1)
+				)
+				(path "/6deb7572-40fc-4be3-9f80-b7a356c09b38/97176d4a-f469-4b3e-946d-de72b475fa7f"
+					(reference "#PWR0248")
+					(unit 1)
+				)
+				(path "/6deb7572-40fc-4be3-9f80-b7a356c09b38/bb90eeae-f6b7-4ab0-91ca-1f494e8dc0e5"
+					(reference "#PWR0230")
+					(unit 1)
+				)
 			)
 		)
@@
 					(unit 1)
 				)
+				(path "/6deb7572-40fc-4be3-9f80-b7a356c09b38/8c1e6824-86fa-49c6-92ab-5b5974896eb4"
+					(reference "#PWR0255")
+					(unit 1)
+				)
+				(path "/6deb7572-40fc-4be3-9f80-b7a356c09b38/97176d4a-f469-4b3e-946d-de72b475fa7f"
+					(reference "#PWR0247")
+					(unit 1)
+				)
+				(path "/6deb7572-40fc-4be3-9f80-b7a356c09b38/bb90eeae-f6b7-4ab0-91ca-1f494e8dc0e5"
+					(reference "#PWR0229")
+					(unit 1)
+				)
 			)
 		)
@@
 					(unit 1)
 				)
+				(path "/6deb7572-40fc-4be3-9f80-b7a356c09b38/8c1e6824-86fa-49c6-92ab-5b5974896eb4"
+					(reference "D37")
+					(unit 1)
+				)
+				(path "/6deb7572-40fc-4be3-9f80-b7a356c09b38/97176d4a-f469-4b3e-946d-de72b475fa7f"
+					(reference "D26")
+					(unit 1)
+				)
+				(path "/6deb7572-40fc-4be3-9f80-b7a356c09b38/bb90eeae-f6b7-4ab0-91ca-1f494e8dc0e5"
+					(reference "D23")
+					(unit 1)
+				)
 			)
 		)
@@
 					(unit 1)
 				)
+				(path "/6deb7572-40fc-4be3-9f80-b7a356c09b38/8c1e6824-86fa-49c6-92ab-5b5974896eb4"
+					(reference "#PWR0253")
+					(unit 1)
+				)
+				(path "/6deb7572-40fc-4be3-9f80-b7a356c09b38/97176d4a-f469-4b3e-946d-de72b475fa7f"
+					(reference "#PWR0245")
+					(unit 1)
+				)
+				(path "/6deb7572-40fc-4be3-9f80-b7a356c09b38/bb90eeae-f6b7-4ab0-91ca-1f494e8dc0e5"
+					(reference "#PWR0227")
+					(unit 1)
+				)
 			)
 		)
@@
 					(unit 1)
 				)
+				(path "/6deb7572-40fc-4be3-9f80-b7a356c09b38/8c1e6824-86fa-49c6-92ab-5b5974896eb4"
+					(reference "R92")
+					(unit 1)
+				)
+				(path "/6deb7572-40fc-4be3-9f80-b7a356c09b38/97176d4a-f469-4b3e-946d-de72b475fa7f"
+					(reference "R84")
+					(unit 1)
+				)
+				(path "/6deb7572-40fc-4be3-9f80-b7a356c09b38/bb90eeae-f6b7-4ab0-91ca-1f494e8dc0e5"
+					(reference "R76")
+					(unit 1)
+				)
 			)
 		)
@@
 					(unit 1)
 				)
+				(path "/6deb7572-40fc-4be3-9f80-b7a356c09b38/8c1e6824-86fa-49c6-92ab-5b5974896eb4"
+					(reference "R87")
+					(unit 1)
+				)
+				(path "/6deb7572-40fc-4be3-9f80-b7a356c09b38/97176d4a-f469-4b3e-946d-de72b475fa7f"
+					(reference "R79")
+					(unit 1)
+				)
+				(path "/6deb7572-40fc-4be3-9f80-b7a356c09b38/bb90eeae-f6b7-4ab0-91ca-1f494e8dc0e5"
+					(reference "R71")
+					(unit 1)
+				)
 			)
 		)
@@
 					(unit 1)
 				)
+				(path "/6deb7572-40fc-4be3-9f80-b7a356c09b38/8c1e6824-86fa-49c6-92ab-5b5974896eb4"
+					(reference "C45")
+					(unit 1)
+				)
+				(path "/6deb7572-40fc-4be3-9f80-b7a356c09b38/97176d4a-f469-4b3e-946d-de72b475fa7f"
+					(reference "C42")
+					(unit 1)
+				)
+				(path "/6deb7572-40fc-4be3-9f80-b7a356c09b38/bb90eeae-f6b7-4ab0-91ca-1f494e8dc0e5"
+					(reference "C39")
+					(unit 1)
+				)
 			)
 		)
@@
 					(unit 1)
 				)
+				(path "/6deb7572-40fc-4be3-9f80-b7a356c09b38/8c1e6824-86fa-49c6-92ab-5b5974896eb4"
+					(reference "#PWR0254")
+					(unit 1)
+				)
+				(path "/6deb7572-40fc-4be3-9f80-b7a356c09b38/97176d4a-f469-4b3e-946d-de72b475fa7f"
+					(reference "#PWR0246")
+					(unit 1)
+				)
+				(path "/6deb7572-40fc-4be3-9f80-b7a356c09b38/bb90eeae-f6b7-4ab0-91ca-1f494e8dc0e5"
+					(reference "#PWR0228")
+					(unit 1)
+				)
 			)
 		)
@@
 					(unit 1)
 				)
+				(path "/6deb7572-40fc-4be3-9f80-b7a356c09b38/8c1e6824-86fa-49c6-92ab-5b5974896eb4"
+					(reference "C44")
+					(unit 1)
+				)
+				(path "/6deb7572-40fc-4be3-9f80-b7a356c09b38/97176d4a-f469-4b3e-946d-de72b475fa7f"
+					(reference "C41")
+					(unit 1)
+				)
+				(path "/6deb7572-40fc-4be3-9f80-b7a356c09b38/bb90eeae-f6b7-4ab0-91ca-1f494e8dc0e5"
+					(reference "C38")
+					(unit 1)
+				)

Commit message: started pin assignement
Parts:
- removed R15, R5: 10k, symbol Device:R
- removed R16, R6: 20k, symbol Device:R
- removed R4, R7: 4k7, symbol Device:R
- added R38, R41: 4.7kΩ, PCM_JLCPCB:R_0805, symbol PCM_JLCPCB-Resistors:0805,4.7kΩ
- added R39, R42: 10kΩ, PCM_JLCPCB:R_0805, symbol PCM_JLCPCB-Resistors:0805,10kΩ
- added R40, R43: 20kΩ, PCM_JLCPCB:R_0805, symbol PCM_JLCPCB-Resistors:0805,20kΩ
- renumbered C2 to C60, C4 to C61, D2 to D5, D3 to D6
Connections:
- net +5V: now also R38.1, R41.1
- net GND: now also R40.2, R43.2
- net MCU_PAS_A: now also R39.2, R40.1
- net MCU_PAS_B: now also R42.2, R43.1
- net PAS_A: now also R38.2, R39.1
- net PAS_B: now also R41.2, R42.1
