File: MCU.kicad_sch (KiCad schematic)
At the start: 0 parts

Commit message: MCU+CAN
Parts:
- added C247, C250, C256, C257, C258, C260, C261, C262, C263, C264, C265, C266, C267, C268, C271, C284, C285, C292, C321: 0u1, Capacitor_SMD:C_0603_1608Metric, symbol Device:C
- added C248, C249: 18p, Capacitor_SMD:C_0402_1005Metric, symbol Device:C
- added C251, C259: 10u/16V/X7R, Capacitor_SMD:C_0805_2012Metric, symbol Device:C
- added C269, C270: 12p, Capacitor_SMD:C_0603_1608Metric, symbol Device:C
- added C282, C283: 2u2/16V/X7R, Capacitor_SMD:C_0805_2012Metric, symbol Device:C
- added J4: Conn_01x06_Pin, Connector_PinHeader_2.00mm:PinHeader_2x03_P2.00mm_Vertical_SMD, symbol Connector:Conn_01x06_Pin
- added L24: 10u/450mA, Inductor_SMD:L_1210_3225Metric, symbol Device:L_Ferrite
- added R208: 10k, Resistor_SMD:R_0603_1608Metric, symbol Device:R
- added R209, R210, R211, R212, R216, R217, R218, R219, R263, R264: 2k2, Resistor_SMD:R_0603_1608Metric, symbol Device:R
- added R220, R226, R227, R228, R233, R234: 0R, Resistor_SMD:R_0603_1608Metric, symbol Device:R
- added TP12: SWCLK, TestPoint:TestPoint_Pad_D1.5mm, symbol Connector:TestPoint
- added TP13: SWDIO, TestPoint:TestPoint_Pad_D1.5mm, symbol Connector:TestPoint
- added TP14: ~{ucRST}, TestPoint:TestPoint_Pad_D1.5mm, symbol Connector:TestPoint
- added TP2: MEM_WP, TestPoint:TestPoint_THTPad_D1.5mm_Drill0.7mm, symbol Connector:TestPoint
- added TP28: BOOT, TestPoint:TestPoint_Pad_D1.5mm, symbol Connector:TestPoint
- added U1: STM32H723ZGT6, Package_QFP:LQFP-144_20x20mm_P0.5mm, symbol MCU_ST_STM32H7:STM32H723ZGTx
- added U51: 24AA02-OT, Package_TO_SOT_SMD:SOT-23-5, symbol Memory_EEPROM:24AA02-OT
- added Y5: 12M, Crystal:Crystal_SMD_Abracon_ABM8G-4Pin_3.2x2.5mm, symbol Device:Crystal_GND24
- added Y6: 32,768kHz, Crystal:Crystal_SMD_EuroQuartz_EQ161-2Pin_3.2x1.5mm, symbol Device:Crystal
Connections:
- new net: R227.2, R228.2, U1.143 (PDR_ON)
- new net: R233.1, R234.2, U1.6 (VBAT)
- new net: C282.1, C283.1, C284.1, C285.1, U1.106 (VCAP), U1.71 (VCAP)
- new net: R220.2, R226.2, TP28.1, U1.138 (BOOT0)
- new net: R263.2, R264.1, TP2.1, U51.5 (WP)
- new net: C248.1, U1.23 (PH0), Y5.1
- new net: C249.1, Y5.3
- new net +3.3V: C250.1, C251.1, C256.1, C257.1, C258.1, C261.1, C262.1, C263.1, C264.1, C265.1, C266.1, C267.1, C268.1, C292.1, C321.1, J4.1 (Pin_1), L24.1, R208.1, R209.1, R210.1, R211.1, R212.1, R216.1, R217.1, R218.1, R219.1, R226.1, R227.1, R233.2, R263.1, U1.108 (VDD), U1.121 (VDD), U1.131 (VDD), U1.144 (VDD), U1.17 (VDD), U1.30 (VDD), U1.39 (VDD), U1.52 (VDD), U1.62 (VDD), U1.72 (VDD), U1.84 (VDD), U1.95 (VDD33USB), U51.4 (V_{CC})
- new net +3.3VA: C259.1, C260.1, C271.1, L24.2, U1.32 (VREF+), U1.33 (VDDA)
- new net +VBAT: R234.1
- new net GND: C247.2, C248.2, C249.2, C250.2, C251.2, C256.2, C257.2, C258.2, C259.2, C260.2, C261.2, C262.2, C263.2, C264.2, C265.2, C266.2, C267.2, C268.2, C269.2, C270.2, C271.2, C282.2, C283.2, C284.2, C285.2, C292.2, C321.2, J4.5 (Pin_5), R220.1, R228.1, R264.2, U1.107 (VSS), U1.120 (VSS), U1.130 (VSS), U1.16 (VSS), U1.31 (VSSA), U1.38 (VSS), U1.51 (VSS), U1.61 (VSS), U1.83 (VSS), U1.94 (VSS), U51.2 (V_{SS}), Y5.2, Y5.4
- new net I2C1.CLK: R209.2
- new net I2C1.DATA: R210.2
- new net I2C2.DATA: R212.2, U51.1 (SCL)
- new net I2C2.SCK: R211.2, U51.3 (SDA)
- new net I2C4.DATA: R217.2
- new net I2C4.INT1: R219.2
- new net I2C4.INT2: R218.2
- new net I2C4.SCK: R216.2
- new net SW0.SWCLK: J4.2 (Pin_2), TP12.1, U1.109 (PA14(JTCK)
- new net SW0.SWDIO: J4.3 (Pin_3), TP13.1, U1.105 (PA13(JTMS)
- new net SW0.SWO: J4.6 (Pin_6)
- new net SW0.~{ucRST}: C247.1, J4.4 (Pin_4), R208.2, TP14.1, U1.25 (NRST)
Changed lines of the file:
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@@
 	(generator_version "10.0")
 	(paper "A4")
-)

Commit message: Integration of changes into prewious style of schematic
Connections:
- net at Y6.1: now also C269.1, U1.9 (PC15)
- net at Y6.2: now also C270.1, U1.8 (PC14)

Commit message: IMU block implementation
Connections:
- net at C270.1, U1.8 (PC14): no longer Y6.2

Commit message: EMI/EMC meassures implementation + VCU panel interface block
Parts:
- C247, C248, C249, C250, C251, C256, C257, C258, C259, C260, C261, C262, C263, C264, C265, C266, C267, C268, C269, C270, C271, C282, C283, C284, C285, C292, C321: symbol Device:C -> VELION_VCU_Library:C
- J4: symbol Connector:Conn_01x06_Pin -> VELION_VCU_Library:Conn_01x06_Pin
- L24: symbol Device:L_Ferrite -> VELION_VCU_Library:L_Ferrite
- R208, R209, R210, R211, R212, R216, R217, R218, R219, R220, R226, R227, R228, R233, R234, R263, R264: symbol Device:R -> VELION_VCU_Library:R
- TP12, TP13, TP14, TP2, TP28: symbol Connector:TestPoint -> VELION_VCU_Library:TestPoint
- U1: symbol MCU_ST_STM32H7:STM32H723ZGTx -> VELION_VCU_Library:STM32H723ZGTx_2
- U1: symbol MCU_ST_STM32H7:STM32H723ZGTx -> VELION_VCU_Library:STM32H723ZGTx_1
- U1: symbol MCU_ST_STM32H7:STM32H723ZGTx -> VELION_VCU_Library:STM32H723ZGTx_4
- U1: symbol MCU_ST_STM32H7:STM32H723ZGTx -> VELION_VCU_Library:STM32H723ZGTx
- U1: symbol MCU_ST_STM32H7:STM32H723ZGTx -> VELION_VCU_Library:STM32H723ZGTx_3
- U51: symbol Memory_EEPROM:24AA02-OT -> VELION_VCU_Library:24AA02-OT
- Y5: symbol Device:Crystal_GND24 -> VELION_VCU_Library:Crystal_GND24
- Y6: symbol Device:Crystal -> VELION_VCU_Library:Crystal
