File: SideIndicatorLightsControl.kicad_sch (KiCad schematic)
At the start: 15 parts, among them U15 VND7050AJTR, U8 VND7050AJTR

Commit message: I/O Schematic rebuild from DRAFT by Nathann
Parts:
- U15, U8: footprint easyeda2kicad:POWERSSO-16_L4.9-W3.9-P0.50-LS6.0-BL-EP -> Package_SO:PowerSSO-16-1EP_3.9x4.9mm_P0.5mm_EP2.5x3.61mm
Connections:
- net SideMarkLampRightOUT: now reaches J6.2, U8.13 (OUTPUT0), U8.14 (OUTPUT0), U8.15 (OUTPUT0), U8.16 (OUTPUT0)
- net SideDirLampRightOUT: now reaches J6.3, U8.10 (OUTPUT1), U8.11 (OUTPUT1), U8.12 (OUTPUT1), U8.9 (OUTPUT1)
- net SideDirLampLeftOUT: now reaches J11.3, U15.10 (OUTPUT1), U15.11 (OUTPUT1), U15.12 (OUTPUT1), U15.9 (OUTPUT1)
- net SideMarkLampLeftOUT: now reaches J11.2, U15.13 (OUTPUT0), U15.14 (OUTPUT0), U15.15 (OUTPUT0), U15.16 (OUTPUT0)
- net SEL0 renamed SideSEL0
- net SEL1 renamed SideSEL1
- net Sense renamed SideSense
- net output10 renamed SideMarkLampL
- net output11 renamed SideDirLampL
- net output8 renamed SideMarkLampR
- net output9 renamed SideDirLampR
Changed lines of the file:
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@@
 		)
 	)
-	(hierarchical_label "SEL1"
+	(label "SideMarkLampLeftOUT"
+		(at 193.04 71.12 0)
+		(effects
+			(font
+				(size 1.27 1.27)
+			)
+			(justify left bottom)
+		)
+	)
+	(label "SideMarkLampRightOUT"
+		(at 193.04 35.56 0)
+		(effects
+			(font
+				(size 1.27 1.27)
+			)
+			(justify left bottom)
+		)
+	)
+	(label "SideDirLampRightOUT"
+		(at 193.04 38.1 0)
+		(effects
+			(font
+				(size 1.27 1.27)
+			)
+			(justify left bottom)
+		)
+	)
+	(label "SideDirLampLeftOUT"
+		(at 193.04 73.66 0)
+		(effects
+			(font
+				(size 1.27 1.27)
+			)
+			(justify left bottom)
+		)
+	)
+	(hierarchical_label "SideSEL1"
 		(shape input)
 		(at 66.04 119.38 180)
@@
 		)
 	)
-	(hierarchical_label "SEL0"
+	(hierarchical_label "SideSEL0"
 		(shape input)
 		(at 66.04 115.57 180)
@@
 		)
 	)
-	(hierarchical_label "output8"
+	(hierarchical_label "SideMarkLampR"
 		(shape input)
 		(at 92.71 31.75 180)
@@
 		)
 	)
-	(hierarchical_label "Sense"
+	(hierarchical_label "SideSense"
 		(shape output)
 		(at 66.04 125.73 180)
@@
 		)
 	)
-	(hierarchical_label "output9"
+	(hierarchical_label "SideDirLampR"
 		(shape input)
 		(at 92.71 49.53 180)
@@
 		)
 	)
-	(hierarchical_label "output11"
+	(hierarchical_label "SideDirLampL"
 		(shape input)
 		(at 92.71 82.55 180)
@@
 		)
 	)
-	(hierarchical_label "output10"
+	(hierarchical_label "SideMarkLampL"
 		(shape input)
 		(at 92.71 64.77 180)
@@
 			)
 		)
-		(property "Footprint" "easyeda2kicad:POWERSSO-16_L4.9-W3.9-P0.50-LS6.0-BL-EP"
+		(property "Footprint" "Package_SO:PowerSSO-16-1EP_3.9x4.9mm_P0.5mm_EP2.5x3.61mm"
 			(at 128.27 57.15 0)
 			(hide yes)
@@
 			)
 		)
-		(property "Footprint" "easyeda2kicad:POWERSSO-16_L4.9-W3.9-P0.50-LS6.0-BL-EP"
+		(property "Footprint" "Package_SO:PowerSSO-16-1EP_3.9x4.9mm_P0.5mm_EP2.5x3.61mm"
 			(at 128.27 90.17 0)
 			(hide yes)

Commit message: EMI/EMC meassures implementation + VCU panel interface block
Parts:
- added C10, C11, C12, C9: 1n, Capacitor_SMD:C_0603_1608Metric, symbol VELION_VCU_Library:C
- added R65, R66, R67, R68: 22R, Resistor_SMD:R_0603_1608Metric, symbol VELION_VCU_Library:R
- added R69, R70, R71, R72, R73, R74: 1k, Resistor_SMD:R_0603_1608Metric, symbol VELION_VCU_Library:R
- C51, C52: footprint PCM_JLCPCB:C_0805 -> Capacitor_SMD:C_0603_1608Metric; symbol PCM_JLCPCB-Capacitors:0805,100nF,(2) -> VELION_VCU_Library:0805,100nF,(2)
- D12: footprint PCM_JLCPCB:D_SOD-123 -> Diode_SMD:D_SOD-123; symbol PCM_JLCPCB-Diodes:Switching,1N4148W -> VELION_VCU_Library:Switching,1N4148W
- D13: footprint PCM_JLCPCB:SOT-23-3_L2.9-W1.3-P1.90-LS2.4-BR -> Package_TO_SOT_SMD:SOT-23-3; symbol PCM_JLCPCB-Diode-Packages:Schottky, BAT54S_C7420333 -> VELION_VCU_Library:Schottky, BAT54S_C7420333
- J11: symbol JST_JWPF:B04B-JWPF-SK-R -> VELION_VCU_Library:B04B-JWPF-SK-R
- J6: symbol JST_JWPF:B03B-JWPF-SK-R -> VELION_VCU_Library:B03B-JWPF-SK-R
- R33: footprint PCM_JLCPCB:R_0805 -> Resistor_SMD:R_0805_2012Metric; symbol PCM_JLCPCB-Resistors:0805,4.7kΩ -> VELION_VCU_Library:0805,4.7kΩ
- R34, R35, R36, R37, R38, R39: footprint PCM_JLCPCB:R_0805 -> Resistor_SMD:R_0805_2012Metric; symbol PCM_JLCPCB-Resistors:0805,1kΩ -> VELION_VCU_Library:0805,1kΩ
- U15, U8: symbol easyeda2kicad:VND7050AJTR -> VELION_VCU_Library:VND7050AJTR
Connections:
- net GND: now also C10.2, C11.2, C12.2, C9.2
- net SideDirLampL: now also R73.1; no longer U15.8 (INPUT1)
- net SideDirLampLeftOUT: now also R67.1
- net SideDirLampR: now also R70.1; no longer U8.8 (INPUT1)
- net SideDirLampRightOUT: now also R65.1
- net SideMarkLampL: now also R72.1; no longer U15.1 (INPUT0)
- net SideMarkLampLeftOUT: now also R68.1
- net SideMarkLampR: now also R69.1; no longer U8.1 (INPUT0)
- net SideMarkLampRightOUT: now also R66.1
- net selE: now also R71.1; no longer U8.3 (SEn)
- net selF: now also R74.1; no longer U15.3 (SEn)
- new net: C12.1, R68.2
- new net: R70.2, U8.8 (INPUT1)
- new net: R72.2, U15.1 (INPUT0)
- new net: C9.1, R65.2
- new net: C11.1, R67.2
- new net: R74.2, U15.3 (SEn)
- new net: R69.2, U8.1 (INPUT0)
- new net: R71.2, U8.3 (SEn)
- new net: R73.2, U15.8 (INPUT1)
- new net: C10.1, R66.2
Other:
- moved on the sheet: C51, C52, J11, J6
